File: hardware/phase2-module/disconnect.kicad_sch (KiCad schematic)
At the start: 18 parts, among them Q10 CSD18540Q5B, Q11 CSD18540Q5B, Q3 CSD18540Q5B, Q4 CSD18540Q5B, Q7 2N7002, Q9 2N7002, U6 LTC7004, U7 TLV7011

Commit message: Apply China-sourcing engineering changes across all boards + mechanical frame
All datasheet-verified before application (details hardware/SOURCING.md sF):
- TMUX1101 -> TS5A3166DBVR (LCSC availability; ts5a3166.pdf: pin POSITIONS
  identical - 1=NO 2=COM 3=GND 4=IN 5=V+; VIH 2.4V ok from 3.3V GPIO)
- TLV7011 DBVR -> DCKR: tlv7022.pdf shows DBV/DCK share one pinout, so
  footprint-only (SOT-353_SC-70-5); SOT-23-5 stock in China is nearly gone
- crystal load caps 10p -> 18p, both phases (CL=12pF China crystals; the
  HANDOVER-blessed alternative to hunting CL=8pF parts)
- Phase-1 inductor -> MWSA1707S-100MT (JLCPCB-verified 16.5A Isat/10.5A
  Irms vs 12A/8A required); value strings now dual-source Sunlord/Coilcraft
- module slot power + P2 output -> XT60PW-M (2-pin), backplane slots ->
  XT60PW-F; bus shunt -> 2x BVS-M-R0005 parallel (the exact-net checker
  caught RS1/RS2 placed one pin-span apart merging VBUS_IN into VBUS)
- 470u bulk -> THT radial D10; output MLCCs 22u -> 10u/50V X7S; buzzer ->
  MLT-8530 (fp placeholder)
All four checker chains green: 137/173/30/80 components.

hardware/MECHANICAL.md (frozen): 30mm slot pitch, P2 130x90 4-layer,
backplane ~330x100 2-layer 2oz, manager 100x80; cost-first stackup (1oz
outer + solder-reinforced bus, 2oz only if the thermal soak demands it);
inductor footprint = SUPERSET pattern accepting Sunlord 1707 AND Coilcraft
XAL1510 so the A/B pair is a pure part swap.

HANDOVER: sub-0.5V mV-accurate output DEFERRED to a future dedicated
linear post-regulator module (user decision 2026-07-18); buck floors
documented (P2 0.7V @30V bus, P1 0.5V).

Co-Authored-By: Claude Fable 5 <noreply@anthropic.com>
Parts:
- U7: value TLV7011 -> TLV7011DCK; footprint Package_TO_SOT_SMD:SOT-23-5 -> Package_TO_SOT_SMD:SOT-353_SC-70-5
Changed lines of the file:
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@@
     (in_bom yes) (on_board yes) (dnp no)
     (property "Reference" "U7" (at 165.1 123.19 0) (effects (font (size 1.27 1.27))))
-    (property "Value" "TLV7011" (at 165.1 135.89000000000001 0) (effects (font (size 1.27 1.27))))
-    (property "Footprint" "Package_TO_SOT_SMD:SOT-23-5" (at 165.1 127.0 0) (effects (font (size 1.27 1.27)) hide))
+    (property "Value" "TLV7011DCK" (at 165.1 135.89000000000001 0) (effects (font (size 1.27 1.27))))
+    (property "Footprint" "Package_TO_SOT_SMD:SOT-353_SC-70-5" (at 165.1 127.0 0) (effects (font (size 1.27 1.27)) hide))
     (property "Datasheet" "~" (at 165.1 127.0 0) (effects (font (size 1.27 1.27)) hide))
     (pin "1")
