File: hardware/phase2-module/disconnect.kicad_sch (KiCad schematic)
At the start: 18 parts, among them Q10 CSD18540Q5B, Q11 CSD18540Q5B, Q3 CSD18540Q5B, Q4 CSD18540Q5B, Q7 2N7002, Q9 2N7002, U6 LTC7004, U7 TLV7011DCK

Commit message: Add LCSC part numbers to all four boards' schematics and generate BOMs
common/bom.py writes hidden LCSC/MPN/Manufacturer properties into the
placed symbols (additive only, both one-line and KiCad multi-line
property styles) and emits <board>/bom/<board>-bom.csv plus a
JLCPCB-format CSV. Part table in common/lcsc_parts.py, transcribed
from SOURCING.md with explicit references per board; CHECK notes flag
footprint/variant mismatches. --check fails on stale output.

Co-Authored-By: Claude Opus 5.5 (1M context) <noreply@anthropic.com>
Claude-Session: https://claude.ai/code/session_01MKtKgebN9BpUrgqHq9t7pT
Parts:
- D8: LCSC (none) -> C41283; MPN (none) -> TL431BIDBZR; Manufacturer (none) -> TI
- Q10, Q11, Q3, Q4: LCSC (none) -> C86513; MPN (none) -> CSD18540Q5B; Manufacturer (none) -> TI
- U6: LCSC (none) -> C690105; MPN (none) -> LTC7004EMSE#PBF; Manufacturer (none) -> ADI
- U7: LCSC (none) -> C193688; MPN (none) -> TLV7011DCKR; Manufacturer (none) -> TI
Changed lines of the file:
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@@
+      (effects (font (size 1.27 1.27)) hide)
+    )
+    (property "LCSC" "C86513" (at 93.98 68.58 0)
+      (effects (font (size 1.27 1.27)) hide)
+    )
+    (property "MPN" "CSD18540Q5B" (at 93.98 68.58 0)
+      (effects (font (size 1.27 1.27)) hide)
+    )
+    (property "Manufacturer" "TI" (at 93.98 68.58 0)
       (effects (font (size 1.27 1.27)) hide)
     )
@@
     )
     (property "Datasheet" "~" (at 113.03 102.87 0)
+      (effects (font (size 1.27 1.27)) hide)
+    )
+    (property "LCSC" "C690105" (at 113.03 102.87 0)
+      (effects (font (size 1.27 1.27)) hide)
+    )
+    (property "MPN" "LTC7004EMSE#PBF" (at 113.03 102.87 0)
+      (effects (font (size 1.27 1.27)) hide)
+    )
+    (property "Manufacturer" "ADI" (at 113.03 102.87 0)
       (effects (font (size 1.27 1.27)) hide)
     )
@@
       (effects (font (size 1.27 1.27)) hide)
     )
+    (property "LCSC" "C86513" (at 66.04 35.56 0)
+      (effects (font (size 1.27 1.27)) hide)
+    )
+    (property "MPN" "CSD18540Q5B" (at 66.04 35.56 0)
+      (effects (font (size 1.27 1.27)) hide)
+    )
+    (property "Manufacturer" "TI" (at 66.04 35.56 0)
+      (effects (font (size 1.27 1.27)) hide)
+    )
     (pin "1")
     (pin "2")
@@
       (effects (font (size 1.27 1.27)) hide)
     )
+    (property "LCSC" "C86513" (at 64.77 68.58 0)
+      (effects (font (size 1.27 1.27)) hide)
+    )
+    (property "MPN" "CSD18540Q5B" (at 64.77 68.58 0)
+      (effects (font (size 1.27 1.27)) hide)
+    )
+    (property "Manufacturer" "TI" (at 64.77 68.58 0)
+      (effects (font (size 1.27 1.27)) hide)
+    )
     (pin "1")
     (pin "2")
@@
       (effects (font (size 1.27 1.27)) hide)
     )
+    (property "LCSC" "C86513" (at 95.25 34.29 0)
+      (effects (font (size 1.27 1.27)) hide)
+    )
+    (property "MPN" "CSD18540Q5B" (at 95.25 34.29 0)
+      (effects (font (size 1.27 1.27)) hide)
+    )
+    (property "Manufacturer" "TI" (at 95.25 34.29 0)
+      (effects (font (size 1.27 1.27)) hide)
+    )
     (pin "1")
     (pin "2")
@@
     )
     (property "Datasheet" "~" (at 57.15 100.33 0)
+      (effects (font (size 1.27 1.27)) hide)
+    )
+    (property "LCSC" "C193688" (at 57.15 100.33 0)
+      (effects (font (size 1.27 1.27)) hide)
+    )
+    (property "MPN" "TLV7011DCKR" (at 57.15 100.33 0)
+      (effects (font (size 1.27 1.27)) hide)
+    )
+    (property "Manufacturer" "TI" (at 57.15 100.33 0)
       (effects (font (size 1.27 1.27)) hide)
     )
@@
       (effects (font (size 1.27 1.27)) hide)
     )
+    (property "LCSC" "C41283" (at 206.375 71.755 0)
+      (effects (font (size 1.27 1.27)) hide)
+    )
+    (property "MPN" "TL431BIDBZR" (at 206.375 71.755 0)
+      (effects (font (size 1.27 1.27)) hide)
+    )
+    (property "Manufacturer" "TI" (at 206.375 71.755 0)
+      (effects (font (size 1.27 1.27)) hide)
+    )
