File: hardware/phase2-module/mcu-can.kicad_sch (KiCad schematic)
At the start: 29 parts, among them J2 SWD, J3 UART, U10 STM32G431CBT6, U11 TCAN1042HGV, Y1 8MHz

Commit message: Add LCSC part numbers to all four boards' schematics and generate BOMs
common/bom.py writes hidden LCSC/MPN/Manufacturer properties into the
placed symbols (additive only, both one-line and KiCad multi-line
property styles) and emits <board>/bom/<board>-bom.csv plus a
JLCPCB-format CSV. Part table in common/lcsc_parts.py, transcribed
from SOURCING.md with explicit references per board; CHECK notes flag
footprint/variant mismatches. --check fails on stale output.

Co-Authored-By: Claude Opus 5.5 (1M context) <noreply@anthropic.com>
Claude-Session: https://claude.ai/code/session_01MKtKgebN9BpUrgqHq9t7pT
Parts:
- U10: LCSC (none) -> C529355; MPN (none) -> STM32G431CBT6; Manufacturer (none) -> ST
- U11: LCSC (none) -> C485806; MPN (none) -> TCAN1042VDRQ1; Manufacturer (none) -> TI
- Y1: LCSC (none) -> C400090
Changed lines of the file:
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@@
+      (effects (font (size 1.27 1.27)) hide)
+    )
+    (property "LCSC" "C400090" (at 214.63 130.81 0)
       (effects (font (size 1.27 1.27)) hide)
     )
@@
     )
     (property "Datasheet" "~" (at 139.7 109.22 0)
+      (effects (font (size 1.27 1.27)) hide)
+    )
+    (property "LCSC" "C529355" (at 139.7 109.22 0)
+      (effects (font (size 1.27 1.27)) hide)
+    )
+    (property "MPN" "STM32G431CBT6" (at 139.7 109.22 0)
+      (effects (font (size 1.27 1.27)) hide)
+    )
+    (property "Manufacturer" "ST" (at 139.7 109.22 0)
       (effects (font (size 1.27 1.27)) hide)
     )
@@
       (effects (font (size 1.27 1.27)) hide)
     )
+    (property "LCSC" "C485806" (at 113.03 34.29 0)
+      (effects (font (size 1.27 1.27)) hide)
+    )
+    (property "MPN" "TCAN1042VDRQ1" (at 113.03 34.29 0)
+      (effects (font (size 1.27 1.27)) hide)
+    )
+    (property "Manufacturer" "TI" (at 113.03 34.29 0)
+      (effects (font (size 1.27 1.27)) hide)
+    )

Commit message: Phase-1 BOM: LCSC numbers for every assembled part
Fill the 109 missing Phase-1 placements from the JLCPCB catalogue
(checked 2026-09-27, Basic parts where one fits), so 127 of 136
placements carry an LCSC number. J1-J6 and F1 stay hand-solder;
C17 and R17 are DNP.

Out-of-stock swaps: Q1-Q4 CSD18563Q5A -> NTMFS5C670NLT1G (SO-8FL,
same pinout), P1 U5 INA228AIDGSR -> INA228AQDGSRQ1. Y1 moves to the
CL = 12 pF version of the same crystal (C400090 was the 10 pF one).

Co-Authored-By: Claude Opus 5.5 (1M context) <noreply@anthropic.com>
Claude-Session: https://claude.ai/code/session_013uVohQZFdivAh43gw4mZtf
Parts:
- Y1: LCSC C400090 -> C403948; MPN (none) -> TAXM8M4RFDCET2T; Manufacturer (none) -> Yajingxin
Changed lines of the file:
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@@
       (effects (font (size 1.27 1.27)) hide)
     )
-    (property "LCSC" "C400090" (at 214.63 130.81 0)
+    (property "MPN" "TAXM8M4RFDCET2T" (at 214.63 130.81 0)
       (effects (font (size 1.27 1.27)) hide)
     )
+    (property "Manufacturer" "Yajingxin" (at 214.63 130.81 0)
+      (effects (font (size 1.27 1.27)) hide)
+    )
+    (property "LCSC" "C403948" (at 214.63 130.81 0)
+      (effects (font (size 1.27 1.27)) hide)
+    )
