File: hardware/phase2-module/io.kicad_sch (KiCad schematic)
At the start: 6 parts, among them J1 XT60PW-M SLOT PWR, J4 XT60PW-M OUTPUT, J5 SLOT SIGNALS, J6 FAN, Q8 2N7002

Commit message: Add LCSC part numbers to all four boards' schematics and generate BOMs
common/bom.py writes hidden LCSC/MPN/Manufacturer properties into the
placed symbols (additive only, both one-line and KiCad multi-line
property styles) and emits <board>/bom/<board>-bom.csv plus a
JLCPCB-format CSV. Part table in common/lcsc_parts.py, transcribed
from SOURCING.md with explicit references per board; CHECK notes flag
footprint/variant mismatches. --check fails on stale output.

Co-Authored-By: Claude Opus 5.5 (1M context) <noreply@anthropic.com>
Claude-Session: https://claude.ai/code/session_01MKtKgebN9BpUrgqHq9t7pT
Parts:
- J1, J4: LCSC (none) -> C98732; MPN (none) -> XT60PW-M; Manufacturer (none) -> Amass
Changed lines of the file:
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@@
+      (effects (font (size 1.27 1.27)) hide)
+    )
+    (property "LCSC" "C98732" (at 88.9 81.28 0)
+      (effects (font (size 1.27 1.27)) hide)
+    )
+    (property "MPN" "XT60PW-M" (at 88.9 81.28 0)
+      (effects (font (size 1.27 1.27)) hide)
+    )
+    (property "Manufacturer" "Amass" (at 88.9 81.28 0)
       (effects (font (size 1.27 1.27)) hide)
     )
@@
       (effects (font (size 1.27 1.27)) hide)
     )
+    (property "LCSC" "C98732" (at 87.63 67.31 0)
+      (effects (font (size 1.27 1.27)) hide)
+    )
+    (property "MPN" "XT60PW-M" (at 87.63 67.31 0)
+      (effects (font (size 1.27 1.27)) hide)
+    )
+    (property "Manufacturer" "Amass" (at 87.63 67.31 0)
+      (effects (font (size 1.27 1.27)) hide)
+    )
