File: hardware/phase2-module/phase2-module.kicad_pcb (KiCad board)
At the start: 4 copper layers, 130 x 90 mm, 180 parts, among them J1 XT60PW-M SLOT PWR, J2 SWD, J3 UART, J4 XT60PW-M OUTPUT, J5 SLOT SIGNALS, J6 FAN, Q1 CSD18540Q5B, Q10 CSD18540Q5B, Q11 CSD18540Q5B, Q12 CSD18540Q5B, Q13 CSD18540Q5B, Q14 CSD19536KTT, Q2 CSD18540Q5B, Q3 CSD18540Q5B, Q4 CSD18540Q5B, Q5 2N7002, Q6 2N7002, Q7 2N7002, Q8 2N7002, Q9 2N7002, U1 DAC80502DRXT, U10 STM32G431CBT6, U11 TCAN1042HGV, U12 LM5069MM-2, U13 TS5A3166, U2 OPA2333, U3 LM5143RHAR, U4 INA240A3, U5 INA228, U6 LTC7004, U7 TLV7011DCK, U8 LMR36015AQRNXRQ1, U9 NCP1117-3.3, Y1 8MHz

Commit message: Phase-2 copper pass-1 to 0 DRC; backplane board complete; autorouter
Phase-2 module (130x90 4L):
- route_board.py: clear the last 3 copper clusters (U6 rot-180 stubs,
  U3 gate fan-out incl. the CS2 chain that was attached to pin 3
  instead of pin 4, U5 sense via-on-pad, R32 clip) -> 0 copper DRC,
  0 mask/hole/dangling. 238 unconnected = signal nets for autoroute.
- autoroute.py: phase-1 router with its fix list applied (net-blind
  via hole spacing, plane targets from in1/in2 maps) on a 0.125 mm
  bytearray grid after the 0.25 mm grid proved unable to hit the
  0.185 mm-wide legal lanes at the fine-pitch escapes.

Phase-3 backplane (330x100 2L 2oz): single-script gen_board.py,
fully placed AND routed, 0 copper DRC / 0 unconnected. XT60PW-F at
rot 90 mates the module connector pad-for-pad (same y offsets, socket
row = module J5 1:1); M6 lugs -> RS1||RS2 0.5 mOhm with INA228 Kelvin
tap between the shunts; mirrored 2oz bus bands + stitching; nested
PRESENT L-bus; CAN terminated past both end slots; E-stop chain
threads the NC switch per docs.

HANDOVER.md: resume section updated (copper done, autoroute notes,
backplane state); .gitignore: VSCode .history/ folders.

Co-Authored-By: Claude Fable 5 <noreply@anthropic.com>
Parts:
- moved C32 2.98 mm to (144.0, 74.6), turned to 0 degrees
Routing:
- net 5V0: track 8.98 -> 11.9 mm, vias 8 -> 9
- net AGND: track 24.3 -> 25.7 mm, vias 61 -> 62
- net PH_CS_B: track 47.7 -> 48.9 mm, vias 5 -> 6
- net 3V3: track 31.7 -> 30.8 mm, vias 13 -> 12
- net LTC_BST: track 5.39 -> 5.94 mm
- net VOUT_INT: vias 17 -> 16
