File: hardware/phase2-module/phase2-module.kicad_pcb (KiCad board)
At the start: 4 copper layers, 130 x 90 mm, 180 parts, among them J1 XT60PW-M SLOT PWR, J2 SWD, J3 UART, J4 XT60PW-M OUTPUT, J5 SLOT SIGNALS, J6 FAN, Q1 CSD18540Q5B, Q10 CSD18540Q5B, Q11 CSD18540Q5B, Q12 CSD18540Q5B, Q13 CSD18540Q5B, Q14 CSD19536KTT, Q2 CSD18540Q5B, Q3 CSD18540Q5B, Q4 CSD18540Q5B, Q5 2N7002, Q6 2N7002, Q7 2N7002, Q8 2N7002, Q9 2N7002, U1 DAC80502DRXT, U10 STM32G431CBT6, U11 TCAN1042HGV, U12 LM5069MM-2, U13 TS5A3166, U2 OPA2333, U3 LM5143RHAR, U4 INA240A3, U5 INA228, U6 LTC7004, U7 TLV7011DCK, U8 LMR36015AQRNXRQ1, U9 NCP1117-3.3, Y1 8MHz

Commit message: Refactor code structure for improved readability and maintainability
Routing:
- net AGND: track 25.7 -> 197.8 mm, vias 62 -> 101
- net I_MEAS: track 0.00 -> 123.6 mm, vias 0 -> 3
- net HW_EN: track 0.00 -> 123.6 mm, vias 0 -> 6
- net 5V0: track 11.9 -> 113.5 mm, vias 9 -> 29
- net SLOT_ID0: track 0.00 -> 96.8 mm
- net EAI_INJ: track 0.00 -> 89.2 mm, vias 0 -> 4
- net AUX_PG: track 0.00 -> 86.9 mm, vias 0 -> 6
- net SLOT_ID1: track 0.00 -> 85.8 mm, vias 0 -> 2
- net CAN_STB: track 0.00 -> 85.4 mm, vias 0 -> 3
- net V_MEAS: track 0.00 -> 83.5 mm, vias 0 -> 4
- net 3V3: track 30.8 -> 109.8 mm, vias 12 -> 25
- net EAV_INJ: track 0.00 -> 77.3 mm, vias 0 -> 2
- net NTC_FET: track 0.00 -> 74.6 mm, vias 0 -> 2
- net CAN_TX: track 0.00 -> 72.5 mm, vias 0 -> 2
- net CAN_RX: track 0.00 -> 71.3 mm, vias 0 -> 2
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