File: hardware/phase2-module/sensing.kicad_sch (KiCad schematic)
At the start: 16 parts, among them U13 TS5A3166, U4 INA240A3, U5 INA228

Commit message: Add LCSC part numbers to all four boards' schematics and generate BOMs
common/bom.py writes hidden LCSC/MPN/Manufacturer properties into the
placed symbols (additive only, both one-line and KiCad multi-line
property styles) and emits <board>/bom/<board>-bom.csv plus a
JLCPCB-format CSV. Part table in common/lcsc_parts.py, transcribed
from SOURCING.md with explicit references per board; CHECK notes flag
footprint/variant mismatches. --check fails on stale output.

Co-Authored-By: Claude Opus 5.5 (1M context) <noreply@anthropic.com>
Claude-Session: https://claude.ai/code/session_01MKtKgebN9BpUrgqHq9t7pT
Parts:
- R30, R34: LCSC (none) -> C46634444
- U13: LCSC (none) -> C353035; MPN (none) -> TS5A3166DBVR; Manufacturer (none) -> TI
- U4: LCSC (none) -> C2060584; MPN (none) -> INA240A3DR; Manufacturer (none) -> TI
- U5: LCSC (none) -> C2887910; MPN (none) -> INA228AIDGSR; Manufacturer (none) -> TI
Changed lines of the file:
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@@
+      (effects (font (size 1.27 1.27)) hide)
+    )
+    (property "LCSC" "C2887910" (at 130.81 72.39 0)
+      (effects (font (size 1.27 1.27)) hide)
+    )
+    (property "MPN" "INA228AIDGSR" (at 130.81 72.39 0)
+      (effects (font (size 1.27 1.27)) hide)
+    )
+    (property "Manufacturer" "TI" (at 130.81 72.39 0)
       (effects (font (size 1.27 1.27)) hide)
     )
@@
       (effects (font (size 1.27 1.27)) hide)
     )
+    (property "LCSC" "C353035" (at 76.2 125.73 0)
+      (effects (font (size 1.27 1.27)) hide)
+    )
+    (property "MPN" "TS5A3166DBVR" (at 76.2 125.73 0)
+      (effects (font (size 1.27 1.27)) hide)
+    )
+    (property "Manufacturer" "TI" (at 76.2 125.73 0)
+      (effects (font (size 1.27 1.27)) hide)
+    )
     (pin "1")
     (pin "2")
@@
     )
     (property "Datasheet" "~" (at 78.74 77.47 0)
+      (effects (font (size 1.27 1.27)) hide)
+    )
+    (property "LCSC" "C2060584" (at 78.74 77.47 0)
+      (effects (font (size 1.27 1.27)) hide)
+    )
+    (property "MPN" "INA240A3DR" (at 78.74 77.47 0)
+      (effects (font (size 1.27 1.27)) hide)
+    )
+    (property "Manufacturer" "TI" (at 78.74 77.47 0)
       (effects (font (size 1.27 1.27)) hide)
     )
@@
       (effects (font (size 1.27 1.27)) hide)
     )
+    (property "LCSC" "C46634444" (at 219.71 68.58 0)
+      (effects (font (size 1.27 1.27)) hide)
+    )
     (pin "1")
     (pin "2")
@@
       (effects (font (size 1.27 1.27)) hide)
     )
+    (property "LCSC" "C46634444" (at 219.71 60.96 0)
+      (effects (font (size 1.27 1.27)) hide)
+    )

Commit message: BOM: stocked INA228 grade and 10x10 hybrid caps for phase-2
U5 (phase-2) and the backplane U1 move to INA228AQDGSRQ1, the automotive
grade Phase-1 already uses: same VSSOP-10 pinout and register map, in
stock where the AIDGSR is not. C15/16/36/37 become Panasonic EEHZA1V221P
(D10x10.2, 20 mOhm), which fits the CP_Elec_10x10.5 land; the old D8
pick did not, and SUNCON 35HVH220M+P is noted as the same-land fallback.

Co-Authored-By: Claude Opus 5.5 (1M context) <noreply@anthropic.com>
Claude-Session: https://claude.ai/code/session_01CT7ZUC1wFK39SLj4Qnh9qy
Parts:
- U5: LCSC C2887910 -> C5214669; MPN INA228AIDGSR -> INA228AQDGSRQ1
Changed lines of the file:
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@@
       (effects (font (size 1.27 1.27)) hide)
     )
-    (property "LCSC" "C2887910" (at 130.81 72.39 0)
+    (property "LCSC" "C5214669" (at 130.81 72.39 0)
       (effects (font (size 1.27 1.27)) hide)
     )
-    (property "MPN" "INA228AIDGSR" (at 130.81 72.39 0)
+    (property "MPN" "INA228AQDGSRQ1" (at 130.81 72.39 0)
       (effects (font (size 1.27 1.27)) hide)
     )
