File: hardware/phase2-module/phase2-module.kicad_sch (KiCad schematic)
At the start: 0 parts

Commit message: Add autosaved schematic files for power stage and auxiliary rails in phase2-module
Changed lines of the file:
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@@
-(kicad_sch (version 20230121) (generator kicad_gen)
+(kicad_sch (version 20230121) (generator eeschema)
   (paper "A4")
+  (text "Lab_Bench phase-2 module - 600W two-phase CV/CC module (docs/08).\nGenerated schematic; run tools/gen_phase2.py, never hand-edit.\nControl core / sensing / disconnect / aux / MCU sheets are the verified\nPhase-1 blocks (hardware/common/sheets_common.py) with Phase-2 values."
+    (at 218.44 173.99 0)
+    (effects (font (size 1.27 1.27)))
+  )
   (sheet (at 38.1 38.1) (size 38.1 15.24) (fields_autoplaced)
-    (stroke (width 0.1524) (type solid)) (fill (color 0 0 0 0.0))
-    (property "Sheetname" "hot-swap" (at 38.1 37.300000000000004 0) (effects (font (size 1.27 1.27)) (justify left bottom)))
-    (property "Sheetfile" "hot-swap.kicad_sch" (at 38.1 53.940000000000005 0) (effects (font (size 1.27 1.27)) (justify left top)))
-    (instances (project "phase2-module" (path "/f47c11d2-88b1-4e02-9d3a-7f10a2c50001" (page "2"))))
+    (stroke (width 0.1524) (type solid))
+    (fill (color 0 0 0 0.0000))
+    (property "Sheetname" "hot-swap" (at 38.1 37.3 0)
+      (effects (font (size 1.27 1.27)) (justify left bottom))
+    )
+    (property "Sheetfile" "hot-swap.kicad_sch" (at 38.1 53.94 0)
+      (effects (font (size 1.27 1.27)) (justify left top))
+    )
+    (instances
+      (project "phase2-module"
+        (path "/f47c11d2-88b1-4e02-9d3a-7f10a2c50001" (page "2"))
+      )
+    )
   )
   (sheet (at 88.9 38.1) (size 38.1 15.24) (fields_autoplaced)
-    (stroke (width 0.1524) (type solid)) (fill (color 0 0 0 0.0))
-    (property "Sheetname" "power-stage" (at 88.9 37.300000000000004 0) (effects (font (size 1.27 1.27)) (justify left bottom)))
-    (property "Sheetfile" "power-stage.kicad_sch" (at 88.9 53.940000000000005 0) (effects (font (size 1.27 1.27)) (justify left top)))
-    (instances (project "phase2-module" (path "/f47c11d2-88b1-4e02-9d3a-7f10a2c50001" (page "3"))))
+    (stroke (width 0.1524) (type solid))
+    (fill (color 0 0 0 0.0000))
+    (property "Sheetname" "power-stage" (at 88.9 37.3 0)
+      (effects (font (size 1.27 1.27)) (justify left bottom))
+    )
+    (property "Sheetfile" "power-stage.kicad_sch" (at 88.9 53.94 0)
+      (effects (font (size 1.27 1.27)) (justify left top))
+    )
+    (instances
+      (project "phase2-module"
+        (path "/f47c11d2-88b1-4e02-9d3a-7f10a2c50001" (page "3"))
+      )
+    )
   )
   (sheet (at 139.7 38.1) (size 38.1 15.24) (fields_autoplaced)
-    (stroke (width 0.1524) (type solid)) (fill (color 0 0 0 0.0))
-    (property "Sheetname" "control-core" (at 139.7 37.300000000000004 0) (effects (font (size 1.27 1.27)) (justify left bottom)))
-    (property "Sheetfile" "control-core.kicad_sch" (at 139.7 53.940000000000005 0) (effects (font (size 1.27 1.27)) (justify left top)))
-    (instances (project "phase2-module" (path "/f47c11d2-88b1-4e02-9d3a-7f10a2c50001" (page "4"))))
+    (stroke (width 0.1524) (type solid))
+    (fill (color 0 0 0 0.0000))
+    (property "Sheetname" "control-core" (at 139.7 37.3 0)
+      (effects (font (size 1.27 1.27)) (justify left bottom))
+    )
+    (property "Sheetfile" "control-core.kicad_sch" (at 139.7 53.94 0)
+      (effects (font (size 1.27 1.27)) (justify left top))
+    )
+    (instances
+      (project "phase2-module"
+        (path "/f47c11d2-88b1-4e02-9d3a-7f10a2c50001" (page "4"))
+      )
+    )
   )
   (sheet (at 190.5 38.1) (size 38.1 15.24) (fields_autoplaced)
-    (stroke (width 0.1524) (type solid)) (fill (color 0 0 0 0.0))
-    (property "Sheetname" "sensing" (at 190.5 37.300000000000004 0) (effects (font (size 1.27 1.27)) (justify left bottom)))
-    (property "Sheetfile" "sensing.kicad_sch" (at 190.5 53.940000000000005 0) (effects (font (size 1.27 1.27)) (justify left top)))
-    (instances (project "phase2-module" (path "/f47c11d2-88b1-4e02-9d3a-7f10a2c50001" (page "5"))))
+    (stroke (width 0.1524) (type solid))
+    (fill (color 0 0 0 0.0000))
+    (property "Sheetname" "sensing" (at 190.5 37.3 0)
+      (effects (font (size 1.27 1.27)) (justify left bottom))
+    )
+    (property "Sheetfile" "sensing.kicad_sch" (at 190.5 53.94 0)
+      (effects (font (size 1.27 1.27)) (justify left top))
+    )
+    (instances
+      (project "phase2-module"
+        (path "/f47c11d2-88b1-4e02-9d3a-7f10a2c50001" (page "5"))
+      )
+    )
   )
   (sheet (at 38.1 68.58) (size 38.1 15.24) (fields_autoplaced)
-    (stroke (width 0.1524) (type solid)) (fill (color 0 0 0 0.0))
-    (property "Sheetname" "disconnect" (at 38.1 67.78 0) (effects (font (size 1.27 1.27)) (justify left bottom)))
-    (property "Sheetfile" "disconnect.kicad_sch" (at 38.1 84.41999999999999 0) (effects (font (size 1.27 1.27)) (justify left top)))
-    (instances (project "phase2-module" (path "/f47c11d2-88b1-4e02-9d3a-7f10a2c50001" (page "6"))))
+    (stroke (width 0.1524) (type solid))
+    (fill (color 0 0 0 0.0000))
+    (property "Sheetname" "disconnect" (at 38.1 67.78 0)
+      (effects (font (size 1.27 1.27)) (justify left bottom))
+    )
+    (property "Sheetfile" "disconnect.kicad_sch" (at 38.1 84.42 0)
+      (effects (font (size 1.27 1.27)) (justify left top))
+    )
+    (instances
+      (project "phase2-module"
+        (path "/f47c11d2-88b1-4e02-9d3a-7f10a2c50001" (page "6"))
+      )
+    )
   )
   (sheet (at 88.9 68.58) (size 38.1 15.24) (fields_autoplaced)
-    (stroke (width 0.1524) (type solid)) (fill (color 0 0 0 0.0))
-    (property "Sheetname" "aux-rails" (at 88.9 67.78 0) (effects (font (size 1.27 1.27)) (justify left bottom)))
-    (property "Sheetfile" "aux-rails.kicad_sch" (at 88.9 84.41999999999999 0) (effects (font (size 1.27 1.27)) (justify left top)))
-    (instances (project "phase2-module" (path "/f47c11d2-88b1-4e02-9d3a-7f10a2c50001" (page "7"))))
+    (stroke (width 0.1524) (type solid))
+    (fill (color 0 0 0 0.0000))
+    (property "Sheetname" "aux-rails" (at 88.9 67.78 0)
+      (effects (font (size 1.27 1.27)) (justify left bottom))
+    )
+    (property "Sheetfile" "aux-rails.kicad_sch" (at 88.9 84.42 0)
+      (effects (font (size 1.27 1.27)) (justify left top))
+    )
+    (instances
+      (project "phase2-module"
+        (path "/f47c11d2-88b1-4e02-9d3a-7f10a2c50001" (page "7"))
+      )
+    )
   )
   (sheet (at 139.7 68.58) (size 38.1 15.24) (fields_autoplaced)
-    (stroke (width 0.1524) (type solid)) (fill (color 0 0 0 0.0))
-    (property "Sheetname" "mcu-can" (at 139.7 67.78 0) (effects (font (size 1.27 1.27)) (justify left bottom)))
-    (property "Sheetfile" "mcu-can.kicad_sch" (at 139.7 84.41999999999999 0) (effects (font (size 1.27 1.27)) (justify left top)))
-    (instances (project "phase2-module" (path "/f47c11d2-88b1-4e02-9d3a-7f10a2c50001" (page "8"))))
+    (stroke (width 0.1524) (type solid))
+    (fill (color 0 0 0 0.0000))
+    (property "Sheetname" "mcu-can" (at 139.7 67.78 0)
+      (effects (font (size 1.27 1.27)) (justify left bottom))
+    )
+    (property "Sheetfile" "mcu-can.kicad_sch" (at 139.7 84.42 0)
+      (effects (font (size 1.27 1.27)) (justify left top))
+    )
+    (instances
+      (project "phase2-module"
+        (path "/f47c11d2-88b1-4e02-9d3a-7f10a2c50001" (page "8"))
+      )
+    )
   )
   (sheet (at 190.5 68.58) (size 38.1 15.24) (fields_autoplaced)
-    (stroke (width 0.1524) (type solid)) (fill (color 0 0 0 0.0))
-    (property "Sheetname" "io" (at 190.5 67.78 0) (effects (font (size 1.27 1.27)) (justify left bottom)))
-    (property "Sheetfile" "io.kicad_sch" (at 190.5 84.41999999999999 0) (effects (font (size 1.27 1.27)) (justify left top)))
-    (instances (project "phase2-module" (path "/f47c11d2-88b1-4e02-9d3a-7f10a2c50001" (page "9"))))
+    (stroke (width 0.1524) (type solid))
+    (fill (color 0 0 0 0.0000))
+    (property "Sheetname" "io" (at 190.5 67.78 0)
+      (effects (font (size 1.27 1.27)) (justify left bottom))
+    )
+    (property "Sheetfile" "io.kicad_sch" (at 190.5 84.42 0)
+      (effects (font (size 1.27 1.27)) (justify left top))
+    )
+    (instances
+      (project "phase2-module"
+        (path "/f47c11d2-88b1-4e02-9d3a-7f10a2c50001" (page "9"))
+      )
+    )
   )
-  (text "Lab_Bench phase-2 module - 600W two-phase CV/CC module (docs/08).\nGenerated schematic; run tools/gen_phase2.py, never hand-edit.\nControl core / sensing / disconnect / aux / MCU sheets are the verified\nPhase-1 blocks (hardware/common/sheets_common.py) with Phase-2 values." (at 38.1 139.7 0) (effects (font (size 1.27 1.27))))
-  (sheet_instances (path "/" (page "1")))
+  (sheet_instances
+    (path "/" (page "1"))
+  )
 )
