File: hardware/phase3-backplane/phase3-backplane.kicad_pcb (KiCad board)
At the start: 2 copper layers, 330 x 100 mm, 39 parts, among them J1 MANAGER, J10 SLOT0 XT60PW-F, J11 SLOT1 XT60PW-F, J12 SLOT2 XT60PW-F, J13 SLOT3 XT60PW-F, J14 SLOT4 XT60PW-F, J15 SLOT5 XT60PW-F, J16 SLOT6 XT60PW-F, J17 SLOT7 XT60PW-F, J2 E-STOP NC (jumper if absent), J20 SLOT0 SIG, J21 SLOT1 SIG, J22 SLOT2 SIG, J23 SLOT3 SIG, J24 SLOT4 SIG, J25 SLOT5 SIG, J26 SLOT6 SIG, J27 SLOT7 SIG, J30 VBUS+ LUG M6, J31 RETURN LUG M6, U1 INA228

Commit message: Backplane fab-ready; DRC "benign bookkeeping" was two real bugs
The lib_footprint_issues class everyone has been waving through (39
backplane, 180 phase-2, 144 phase-1) was never one thing, and neither
half was harmless bookkeeping:

 1. The board generators add footprints by name only, leaving the FPID
    library nickname empty. common/fix_fpids.py resolves each item name
    against the project library first, then the system libraries, and
    writes the nickname back (363 resolved across three boards, none
    guessed — unresolved names are reported, never invented).
 2. KiCad's global fp-lib-table expands ${KICAD7_FOOTPRINT_DIR}, which
    only the GUI sets. Headless DRC could not expand a single library
    URI, so every footprint came back "not found in library". Every
    run_drc.py now sets it before importing pcbnew.

Both mattered beyond noise: with the libraries unresolved, KiCad cannot
diff a board footprint against its library, so silent land-pattern drift
would pass unnoticed — and this project already caught one such bug in
LM5143 by hand.

    phase3-backplane   40 -> 0 violations, 0 unconnected
    phase2-module     191 -> 11 (silk only), 83 unconnected
    phase1-module     247 -> 75 (silk only)

phase3-backplane is now FAB-READY: silk reflowed (39/39 refs clean), no
plane islands, gerbers + drills plotted and cross-checked — Edge_Cuts
exactly 330.00 x 100.00 mm, drills 2x6.4mm (M6 entry lugs), 16x2.8mm
(8 slots x 2 XT60 pins), 6x3.2mm (M3), 86x1.0mm, 61x0.4mm.

New shared tooling in hardware/common (was phase-2-only, now serves every
board): layout_qa.py (silk reflow, PS-002 islands, gerber/drill plot with
the layer set read from the board) and finish_board.py as its CLI.

Correction: phase-1 is 187 unconnected, not the 33 in HANDOVER — that
figure came from an autoroute run that was never committed, and its
gitignored drc-report.txt kept showing the stale number. Verified against
the committed board.

Co-Authored-By: Claude Fable 5 <noreply@anth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
Parts:
- C1, C3: footprint C_0603_1608Metric -> Capacitor_SMD:C_0603_1608Metric
- C2: footprint CP_Elec_16x17.5 -> Capacitor_SMD:CP_Elec_16x17.5
- D5: footprint D_SMB -> Diode_SMD:D_SMB
- FID1, FID2, FID3: footprint Fiducial_1mm_Mask2mm -> Fiducial:Fiducial_1mm_Mask2mm
- H1, H2, H3, H4, H5, H6: footprint MountingHole_3.2mm_M3 -> MountingHole:MountingHole_3.2mm_M3
- J1: footprint PinHeader_1x20_P2.54mm_Vertical -> Connector_PinHeader_2.54mm:PinHeader_1x20_P2.54mm_Vertical
- J10, J11, J12, J13, J14, J15, J16, J17: footprint XT60PW-F -> labbench:XT60PW-F
- J2: footprint PinHeader_1x02_P2.54mm_Vertical -> Connector_PinHeader_2.54mm:PinHeader_1x02_P2.54mm_Vertical
- J20, J21, J22, J23, J24, J25, J26, J27: footprint PinHeader_1x08_P2.54mm_Vertical -> Connector_PinHeader_2.54mm:PinHeader_1x08_P2.54mm_Vertical
- J30, J31: footprint MountingHole_6.4mm_M6_Pad_TopBottom -> MountingHole:MountingHole_6.4mm_M6_Pad_TopBottom
- R1, R2, R3: footprint R_0603_1608Metric -> Resistor_SMD:R_0603_1608Metric
- RS1, RS2: footprint R3920_BVS -> labbench:R3920_BVS
- U1: footprint VSSOP-10_3x3mm_P0.5mm -> Package_SO:VSSOP-10_3x3mm_P0.5mm
