File: hardware/phase3-backplane/phase3-backplane.kicad_sch (KiCad schematic)
At the start: 30 parts, among them J1 MANAGER, J10 SLOT0 XT60PW-F, J11 SLOT1 XT60PW-F, J12 SLOT2 XT60PW-F, J13 SLOT3 XT60PW-F, J14 SLOT4 XT60PW-F, J15 SLOT5 XT60PW-F, J16 SLOT6 XT60PW-F, J17 SLOT7 XT60PW-F, J2 E-STOP NC (jumper if absent), J20 SLOT0 SIG, J21 SLOT1 SIG, J22 SLOT2 SIG, J23 SLOT3 SIG, J24 SLOT4 SIG, J25 SLOT5 SIG, J26 SLOT6 SIG, J27 SLOT7 SIG, J30 VBUS+ LUG M6, J31 RETURN LUG M6, U1 INA228

Commit message: Add LCSC part numbers to all four boards' schematics and generate BOMs
common/bom.py writes hidden LCSC/MPN/Manufacturer properties into the
placed symbols (additive only, both one-line and KiCad multi-line
property styles) and emits <board>/bom/<board>-bom.csv plus a
JLCPCB-format CSV. Part table in common/lcsc_parts.py, transcribed
from SOURCING.md with explicit references per board; CHECK notes flag
footprint/variant mismatches. --check fails on stale output.

Co-Authored-By: Claude Opus 5.5 (1M context) <noreply@anthropic.com>
Claude-Session: https://claude.ai/code/session_01MKtKgebN9BpUrgqHq9t7pT
Parts:
- J10, J11, J12, J13, J14, J15, J16, J17: LCSC (none) -> C428722; MPN (none) -> XT60PW-F; Manufacturer (none) -> Amass
- RS1, RS2: LCSC (none) -> C466580; MPN (none) -> BVS-M-R0005; Manufacturer (none) -> Isabellenhuette
- U1: LCSC (none) -> C2887910; MPN (none) -> INA228AIDGSR; Manufacturer (none) -> TI
Changed lines of the file:
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@@
+      (effects (font (size 1.27 1.27)) hide)
+    )
+    (property "LCSC" "C428722" (at 342.9 166.37 0)
+      (effects (font (size 1.27 1.27)) hide)
+    )
+    (property "MPN" "XT60PW-F" (at 342.9 166.37 0)
+      (effects (font (size 1.27 1.27)) hide)
+    )
+    (property "Manufacturer" "Amass" (at 342.9 166.37 0)
       (effects (font (size 1.27 1.27)) hide)
     )
@@
     )
     (property "Datasheet" "~" (at 342.9 90.17 0)
+      (effects (font (size 1.27 1.27)) hide)
+    )
+    (property "LCSC" "C428722" (at 342.9 90.17 0)
+      (effects (font (size 1.27 1.27)) hide)
+    )
+    (property "MPN" "XT60PW-F" (at 342.9 90.17 0)
+      (effects (font (size 1.27 1.27)) hide)
+    )
+    (property "Manufacturer" "Amass" (at 342.9 90.17 0)
       (effects (font (size 1.27 1.27)) hide)
     )
@@
     )
     (property "Datasheet" "~" (at 130.81 62.23 0)
+      (effects (font (size 1.27 1.27)) hide)
+    )
+    (property "LCSC" "C466580" (at 130.81 62.23 0)
+      (effects (font (size 1.27 1.27)) hide)
+    )
+    (property "MPN" "BVS-M-R0005" (at 130.81 62.23 0)
+      (effects (font (size 1.27 1.27)) hide)
+    )
+    (property "Manufacturer" "Isabellenhuette" (at 130.81 62.23 0)
       (effects (font (size 1.27 1.27)) hide)
     )
@@
     )
     (property "Datasheet" "~" (at 162.56 138.43 0)
+      (effects (font (size 1.27 1.27)) hide)
+    )
+    (property "LCSC" "C2887910" (at 162.56 138.43 0)
+      (effects (font (size 1.27 1.27)) hide)
+    )
+    (property "MPN" "INA228AIDGSR" (at 162.56 138.43 0)
+      (effects (font (size 1.27 1.27)) hide)
+    )
+    (property "Manufacturer" "TI" (at 162.56 138.43 0)
       (effects (font (size 1.27 1.27)) hide)
     )
@@
       (effects (font (size 1.27 1.27)) hide)
     )
+    (property "LCSC" "C428722" (at 281.94 90.17 0)
+      (effects (font (size 1.27 1.27)) hide)
+    )
+    (property "MPN" "XT60PW-F" (at 281.94 90.17 0)
+      (effects (font (size 1.27 1.27)) hide)
+    )
+    (property "Manufacturer" "Amass" (at 281.94 90.17 0)
+      (effects (font (size 1.27 1.27)) hide)
+    )
     (pin "1")
     (pin "2")
@@
       (effects (font (size 1.27 1.27)) hide)
     )
+    (property "LCSC" "C466580" (at 144.78 62.23 0)
+      (effects (font (size 1.27 1.27)) hide)
+    )
+    (property "MPN" "BVS-M-R0005" (at 144.78 62.23 0)
+      (effects (font (size 1.27 1.27)) hide)
+    )
+    (property "Manufacturer" "Isabellenhuette" (at 144.78 62.23 0)
+      (effects (font (size 1.27 1.27)) hide)
+    )
     (pin "1")
     (pin "2")
@@
       (effects (font (size 1.27 1.27)) hide)
     )
+    (property "LCSC" "C428722" (at 373.38 166.37 0)
+      (effects (font (size 1.27 1.27)) hide)
+    )
+    (property "MPN" "XT60PW-F" (at 373.38 166.37 0)
+      (effects (font (size 1.27 1.27)) hide)
+    )
+    (property "Manufacturer" "Amass" (at 373.38 166.37 0)
+      (effects (font (size 1.27 1.27)) hide)
+    )
     (pin "1")
     (pin "2")
@@
     )
     (property "Datasheet" "~" (at 281.94 166.37 0)
+      (effects (font (size 1.27 1.27)) hide)
+    )
+    (property "LCSC" "C428722" (at 281.94 166.37 0)
+      (effects (font (size 1.27 1.27)) hide)
+    )
+    (property "MPN" "XT60PW-F" (at 281.94 166.37 0)
+      (effects (font (size 1.27 1.27)) hide)
+    )
+    (property "Manufacturer" "Amass" (at 281.94 166.37 0)
       (effects (font (size 1.27 1.27)) hide)
     )
@@
       (effects (font (size 1.27 1.27)) hide)
     )
+    (property "LCSC" "C428722" (at 312.42 166.37 0)
+      (effects (font (size 1.27 1.27)) hide)
+    )
+    (property "MPN" "XT60PW-F" (at 312.42 166.37 0)
+      (effects (font (size 1.27 1.27)) hide)
+    )
+    (property "Manufacturer" "Amass" (at 312.42 166.37 0)
+      (effects (font (size 1.27 1.27)) hide)
+    )
     (pin "1")
     (pin "2")
@@
       (effects (font (size 1.27 1.27)) hide)
     )
+    (property "LCSC" "C428722" (at 373.38 90.17 0)
+      (effects (font (size 1.27 1.27)) hide)
+    )
+    (property "MPN" "XT60PW-F" (at 373.38 90.17 0)
+      (effects (font (size 1.27 1.27)) hide)
+    )
+    (property "Manufacturer" "Amass" (at 373.38 90.17 0)
+      (effects (font (size 1.27 1.27)) hide)
+    )
     (pin "1")
     (pin "2")
@@
       (effects (font (size 1.27 1.27)) hide)
     )
+    (property "LCSC" "C428722" (at 312.42 90.17 0)
+      (effects (font (size 1.27 1.27)) hide)
+    )
+    (property "MPN" "XT60PW-F" (at 312.42 90.17 0)
+      (effects (font (size 1.27 1.27)) hide)
+    )
+    (property "Manufacturer" "Amass" (at 312.42 90.17 0)
+      (effects (font (size 1.27 1.27)) hide)
+    )

Commit message: BOM: stocked INA228 grade and 10x10 hybrid caps for phase-2
U5 (phase-2) and the backplane U1 move to INA228AQDGSRQ1, the automotive
grade Phase-1 already uses: same VSSOP-10 pinout and register map, in
stock where the AIDGSR is not. C15/16/36/37 become Panasonic EEHZA1V221P
(D10x10.2, 20 mOhm), which fits the CP_Elec_10x10.5 land; the old D8
pick did not, and SUNCON 35HVH220M+P is noted as the same-land fallback.

Co-Authored-By: Claude Opus 5.5 (1M context) <noreply@anthropic.com>
Claude-Session: https://claude.ai/code/session_01CT7ZUC1wFK39SLj4Qnh9qy
Parts:
- U1: LCSC C2887910 -> C5214669; MPN INA228AIDGSR -> INA228AQDGSRQ1
Changed lines of the file:
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@@
       (effects (font (size 1.27 1.27)) hide)
     )
-    (property "LCSC" "C2887910" (at 162.56 138.43 0)
+    (property "LCSC" "C5214669" (at 162.56 138.43 0)
       (effects (font (size 1.27 1.27)) hide)
     )
-    (property "MPN" "INA228AIDGSR" (at 162.56 138.43 0)
+    (property "MPN" "INA228AQDGSRQ1" (at 162.56 138.43 0)
       (effects (font (size 1.27 1.27)) hide)
     )

Commit message: Manager L2 and backplane C2: pick stocked parts, re-route L2 as an ECO
Manager L2 (33u/1.2A aux-buck inductor) had a 1210 land, and no stocked
1210 33 uH is rated above 0.5 A. It is now the 5x5 mm cjiang
FNR5040S330MT (C167973: Isat 1.30 A min, Irms 1.20 A min, 0.244 ohm)
on KiCad's L_Changjiang_FNR5040S land.

Board ECO, no full re-route:
- L2 moves to (18.8, 48.4) so its courtyard clears C54, F1 and C50/C51;
  C54/C55 turn 180 so their 5V0 pads line up with L2's 5V0 pad (one
  straight 0.8 mm run) and their PGND pads are tied and dropped to the
  plane west of C55.
- SW_AUX and the 5V0 head are redrawn locked, matching route_critical.py;
  PRESENT1/4-7 are re-routed round the bigger part by finish_routes.py.
- gen_board.py PLACEMENT and route_critical.py ROUTES carry the same
  change, so a full rebuild reproduces it.
- DRC: 0 unconnected, 0 errors, 4 warnings (was 5). Fab zip, BOM, CPL
  regenerated.

Backplane C2 (470u/50V on CP_Elec_16x17.5): Nichicon UCX1H471MNS1MS
(C462700, 16x16.5, 70 mOhm), which fits the existing land; Panasonic
EEEFK1H471AM (C178551) is the fallback. No board change.

Co-Authored-By: Claude Opus 5.5 (1M context) <noreply@anthropic.com>
Claude-Session: https://claude.ai/code/session_016Wr11AqV5ZRbpysgP42oHy
Parts:
- C2: LCSC (none) -> C462700; MPN (none) -> UCX1H471MNS1MS; Manufacturer (none) -> Nichicon
Changed lines of the file:
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@@
+      (effects (font (size 1.27 1.27)) hide)
+    )
+    (property "LCSC" "C462700" (at 173.99 62.23 0)
+      (effects (font (size 1.27 1.27)) hide)
+    )
+    (property "MPN" "UCX1H471MNS1MS" (at 173.99 62.23 0)
+      (effects (font (size 1.27 1.27)) hide)
+    )
+    (property "Manufacturer" "Nichicon" (at 173.99 62.23 0)
       (effects (font (size 1.27 1.27)) hide)
     )
