File: hardware/phase1-module/control-core.kicad_sch (KiCad schematic)
At the start: 17 parts, among them U1 DAC80502DRXT, U2 OPA2333

Commit message: Add LCSC part numbers to all four boards' schematics and generate BOMs
common/bom.py writes hidden LCSC/MPN/Manufacturer properties into the
placed symbols (additive only, both one-line and KiCad multi-line
property styles) and emits <board>/bom/<board>-bom.csv plus a
JLCPCB-format CSV. Part table in common/lcsc_parts.py, transcribed
from SOURCING.md with explicit references per board; CHECK notes flag
footprint/variant mismatches. --check fails on stale output.

Co-Authored-By: Claude Opus 5.5 (1M context) <noreply@anthropic.com>
Claude-Session: https://claude.ai/code/session_01MKtKgebN9BpUrgqHq9t7pT
Parts:
- U1: LCSC (none) -> C1880990; MPN (none) -> DAC80502DRXR; Manufacturer (none) -> TI
- U2: LCSC (none) -> C19608; MPN (none) -> OPA2333AIDGKR; Manufacturer (none) -> TI
Changed lines of the file:
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@@
     (property "Footprint" "labbench:DAC80502_DRX_WSON-10" (at 50.8 101.6 0) (effects (font (size 1.27 1.27)) hide))
     (property "Datasheet" "~" (at 50.8 101.6 0) (effects (font (size 1.27 1.27)) hide))
+    (property "LCSC" "C1880990" (at 50.8 101.6 0) (effects (font (size 1.27 1.27)) hide))
+    (property "MPN" "DAC80502DRXR" (at 50.8 101.6 0) (effects (font (size 1.27 1.27)) hide))
+    (property "Manufacturer" "TI" (at 50.8 101.6 0) (effects (font (size 1.27 1.27)) hide))
     (pin "1")
     (pin "10")
@@
     (property "Footprint" "Package_SO:VSSOP-8_3.0x3.0mm_P0.65mm" (at 137.16 76.2 0) (effects (font (size 1.27 1.27)) hide))
     (property "Datasheet" "~" (at 137.16 76.2 0) (effects (font (size 1.27 1.27)) hide))
+    (property "LCSC" "C19608" (at 137.16 76.2 0) (effects (font (size 1.27 1.27)) hide))
+    (property "MPN" "OPA2333AIDGKR" (at 137.16 76.2 0) (effects (font (size 1.27 1.27)) hide))
+    (property "Manufacturer" "TI" (at 137.16 76.2 0) (effects (font (size 1.27 1.27)) hide))
     (pin "1")
     (pin "2")
@@
     (property "Footprint" "Package_SO:VSSOP-8_3.0x3.0mm_P0.65mm" (at 137.16 127.0 0) (effects (font (size 1.27 1.27)) hide))
     (property "Datasheet" "~" (at 137.16 127.0 0) (effects (font (size 1.27 1.27)) hide))
+    (property "LCSC" "C19608" (at 137.16 127.0 0) (effects (font (size 1.27 1.27)) hide))
+    (property "MPN" "OPA2333AIDGKR" (at 137.16 127.0 0) (effects (font (size 1.27 1.27)) hide))
+    (property "Manufacturer" "TI" (at 137.16 127.0 0) (effects (font (size 1.27 1.27)) hide))
     (pin "5")
     (pin "6")
@@
     (property "Footprint" "Package_SO:VSSOP-8_3.0x3.0mm_P0.65mm" (at 50.8 154.94 0) (effects (font (size 1.27 1.27)) hide))
     (property "Datasheet" "~" (at 50.8 154.94 0) (effects (font (size 1.27 1.27)) hide))
+    (property "LCSC" "C19608" (at 50.8 154.94 0) (effects (font (size 1.27 1.27)) hide))
+    (property "MPN" "OPA2333AIDGKR" (at 50.8 154.94 0) (effects (font (size 1.27 1.27)) hide))
+    (property "Manufacturer" "TI" (at 50.8 154.94 0) (effects (font (size 1.27 1.27)) hide))
     (pin "4")
     (pin "8")

Commit message: Phase-1 BOM: LCSC numbers for every assembled part
Fill the 109 missing Phase-1 placements from the JLCPCB catalogue
(checked 2026-09-27, Basic parts where one fits), so 127 of 136
placements carry an LCSC number. J1-J6 and F1 stay hand-solder;
C17 and R17 are DNP.

Out-of-stock swaps: Q1-Q4 CSD18563Q5A -> NTMFS5C670NLT1G (SO-8FL,
same pinout), P1 U5 INA228AIDGSR -> INA228AQDGSRQ1. Y1 moves to the
CL = 12 pF version of the same crystal (C400090 was the 10 pF one).

Co-Authored-By: Claude Opus 5.5 (1M context) <noreply@anthropic.com>
Claude-Session: https://claude.ai/code/session_013uVohQZFdivAh43gw4mZtf
Parts:
- C1: LCSC (none) -> C57112; MPN (none) -> 0603B103K500NT; Manufacturer (none) -> FH
- C2: LCSC (none) -> C21122; MPN (none) -> CL10B223KB8NNNC; Manufacturer (none) -> Samsung Electro-Mechanics
- C3, C5: LCSC (none) -> C14663; MPN (none) -> CC0603KRX7R9BB104; Manufacturer (none) -> YAGEO
- C4: LCSC (none) -> C513735; MPN (none) -> CC0603KRX7R9BB154; Manufacturer (none) -> YAGEO
- D1, D2: LCSC (none) -> C77328; MPN (none) -> BAT54W; Manufacturer (none) -> Jiangsu Changjing Electronics Technology Co., Ltd.
- R1: LCSC (none) -> C861257; MPN (none) -> RT0603BRD0725K5L; Manufacturer (none) -> YAGEO
- R2: LCSC (none) -> C110776; MPN (none) -> RT0603BRD071KL; Manufacturer (none) -> YAGEO
- R3, R6: LCSC (none) -> C95204; MPN (none) -> RT0603BRD0710KL; Manufacturer (none) -> YAGEO
- R4: LCSC (none) -> C4216; MPN (none) -> 0603WAF3302T5E; Manufacturer (none) -> UNI-ROYAL
- R5, R8: LCSC (none) -> C23018; MPN (none) -> 0603WAF3901T5E; Manufacturer (none) -> UNI-ROYAL
- R7: LCSC (none) -> C22809; MPN (none) -> 0603WAF1502T5E; Manufacturer (none) -> UNI-ROYAL
Changed lines of the file:
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@@
     (property "Footprint" "Capacitor_SMD:C_0603_1608Metric" (at 81.28 111.76 0) (effects (font (size 1.27 1.27)) hide))
     (property "Datasheet" "~" (at 81.28 111.76 0) (effects (font (size 1.27 1.27)) hide))
+    (property "LCSC" "C513735" (at 81.28 111.76 0) (effects (font (size 1.27 1.27)) hide))
+    (property "MPN" "CC0603KRX7R9BB154" (at 81.28 111.76 0) (effects (font (size 1.27 1.27)) hide))
+    (property "Manufacturer" "YAGEO" (at 81.28 111.76 0) (effects (font (size 1.27 1.27)) hide))
     (pin "1")
     (pin "2")
@@
     (property "Footprint" "Capacitor_SMD:C_0603_1608Metric" (at 40.64 127.0 0) (effects (font (size 1.27 1.27)) hide))
     (property "Datasheet" "~" (at 40.64 127.0 0) (effects (font (size 1.27 1.27)) hide))
+    (property "LCSC" "C14663" (at 40.64 127.0 0) (effects (font (size 1.27 1.27)) hide))
+    (property "MPN" "CC0603KRX7R9BB104" (at 40.64 127.0 0) (effects (font (size 1.27 1.27)) hide))
+    (property "Manufacturer" "YAGEO" (at 40.64 127.0 0) (effects (font (size 1.27 1.27)) hide))
     (pin "1")
     (pin "2")
@@
     (property "Footprint" "Resistor_SMD:R_0603_1608Metric" (at 96.52 78.74 0) (effects (font (size 1.27 1.27)) hide))
     (property "Datasheet" "~" (at 96.52 78.74 0) (effects (font (size 1.27 1.27)) hide))
+    (property "LCSC" "C95204" (at 96.52 78.74 0) (effects (font (size 1.27 1.27)) hide))
+    (property "MPN" "RT0603BRD0710KL" (at 96.52 78.74 0) (effects (font (size 1.27 1.27)) hide))
+    (property "Manufacturer" "YAGEO" (at 96.52 78.74 0) (effects (font (size 1.27 1.27)) hide))
     (pin "1")
     (pin "2")
@@
     (property "Footprint" "Capacitor_SMD:C_0603_1608Metric" (at 106.68 58.42 0) (effects (font (size 1.27 1.27)) hide))
     (property "Datasheet" "~" (at 106.68 58.42 0) (effects (font (size 1.27 1.27)) hide))
+    (property "LCSC" "C57112" (at 106.68 58.42 0) (effects (font (size 1.27 1.27)) hide))
+    (property "MPN" "0603B103K500NT" (at 106.68 58.42 0) (effects (font (size 1.27 1.27)) hide))
+    (property "Manufacturer" "FH" (at 106.68 58.42 0) (effects (font (size 1.27 1.27)) hide))
     (pin "1")
     (pin "2")
@@
     (property "Footprint" "Resistor_SMD:R_0603_1608Metric" (at 132.08 58.42 0) (effects (font (size 1.27 1.27)) hide))
     (property "Datasheet" "~" (at 132.08 58.42 0) (effects (font (size 1.27 1.27)) hide))
+    (property "LCSC" "C4216" (at 132.08 58.42 0) (effects (font (size 1.27 1.27)) hide))
+    (property "MPN" "0603WAF3302T5E" (at 132.08 58.42 0) (effects (font (size 1.27 1.27)) hide))
+    (property "Manufacturer" "UNI-ROYAL" (at 132.08 58.42 0) (effects (font (size 1.27 1.27)) hide))
     (pin "1")
     (pin "2")
@@
     (property "Footprint" "Package_TO_SOT_SMD:SOT-323_SC-70" (at 160.02 76.2 0) (effects (font (size 1.27 1.27)) hide))
     (property "Datasheet" "~" (at 160.02 76.2 0) (effects (font (size 1.27 1.27)) hide))
+    (property "LCSC" "C77328" (at 160.02 76.2 0) (effects (font (size 1.27 1.27)) hide))
+    (property "MPN" "BAT54W" (at 160.02 76.2 0) (effects (font (size 1.27 1.27)) hide))
+    (property "Manufacturer" "Jiangsu Changjing Electronics Technology Co., Ltd." (at 160.02 76.2 0) (effects (font (size 1.27 1.27)) hide))
     (pin "1")
     (pin "2")
@@
     (property "Footprint" "Resistor_SMD:R_0603_1608Metric" (at 182.88 76.2 0) (effects (font (size 1.27 1.27)) hide))
     (property "Datasheet" "~" (at 182.88 76.2 0) (effects (font (size 1.27 1.27)) hide))
+    (property "LCSC" "C23018" (at 182.88 76.2 0) (effects (font (size 1.27 1.27)) hide))
+    (property "MPN" "0603WAF3901T5E" (at 182.88 76.2 0) (effects (font (size 1.27 1.27)) hide))
+    (property "Manufacturer" "UNI-ROYAL" (at 182.88 76.2 0) (effects (font (size 1.27 1.27)) hide))
     (pin "1")
     (pin "2")
@@
     (property "Footprint" "Resistor_SMD:R_0603_1608Metric" (at 96.52 129.54 0) (effects (font (size 1.27 1.27)) hide))
     (property "Datasheet" "~" (at 96.52 129.54 0) (effects (font (size 1.27 1.27)) hide))
+    (property "LCSC" "C95204" (at 96.52 129.54 0) (effects (font (size 1.27 1.27)) hide))
+    (property "MPN" "RT0603BRD0710KL" (at 96.52 129.54 0) (effects (font (size 1.27 1.27)) hide))
+    (property "Manufacturer" "YAGEO" (at 96.52 129.54 0) (effects (font (size 1.27 1.27)) hide))
     (pin "1")
     (pin "2")
@@
     (property "Footprint" "Capacitor_SMD:C_0603_1608Metric" (at 106.68 109.22 0) (effects (font (size 1.27 1.27)) hide))
     (property "Datasheet" "~" (at 106.68 109.22 0) (effects (font (size 1.27 1.27)) hide))
+    (property "LCSC" "C21122" (at 106.68 109.22 0) (effects (font (size 1.27 1.27)) hide))
+    (property "MPN" "CL10B223KB8NNNC" (at 106.68 109.22 0) (effects (font (size 1.27 1.27)) hide))
+    (property "Manufacturer" "Samsung Electro-Mechanics" (at 106.68 109.22 0) (effects (font (size 1.27 1.27)) hide))
     (pin "1")
     (pin "2")
@@
     (property "Footprint" "Resistor_SMD:R_0603_1608Metric" (at 132.08 109.22 0) (effects (font (size 1.27 1.27)) hide))
     (property "Datasheet" "~" (at 132.08 109.22 0) (effects (font (size 1.27 1.27)) hide))
+    (property "LCSC" "C22809" (at 132.08 109.22 0) (effects (font (size 1.27 1.27)) hide))
+    (property "MPN" "0603WAF1502T5E" (at 132.08 109.22 0) (effects (font (size 1.27 1.27)) hide))
+    (property "Manufacturer" "UNI-ROYAL" (at 132.08 109.22 0) (effects (font (size 1.27 1.27)) hide))
     (pin "1")
     (pin "2")
@@
     (property "Footprint" "Package_TO_SOT_SMD:SOT-323_SC-70" (at 160.02 127.0 0) (effects (font (size 1.27 1.27)) hide))
     (property "Datasheet" "~" (at 160.02 127.0 0) (effects (font (size 1.27 1.27)) hide))
+    (property "LCSC" "C77328" (at 160.02 127.0 0) (effects (font (size 1.27 1.27)) hide))
+    (property "MPN" "BAT54W" (at 160.02 127.0 0) (effects (font (size 1.27 1.27)) hide))
+    (property "Manufacturer" "Jiangsu Changjing Electronics Technology Co., Ltd." (at 160.02 127.0 0) (effects (font (size 1.27 1.27)) hide))
     (pin "1")
     (pin "2")
@@
     (property "Footprint" "Resistor_SMD:R_0603_1608Metric" (at 182.88 127.0 0) (effects (font (size 1.27 1.27)) hide))
     (property "Datasheet" "~" (at 182.88 127.0 0) (effects (font (size 1.27 1.27)) hide))
+    (property "LCSC" "C23018" (at 182.88 127.0 0) (effects (font (size 1.27 1.27)) hide))
+    (property "MPN" "0603WAF3901T5E" (at 182.88 127.0 0) (effects (font (size 1.27 1.27)) hide))
+    (property "Manufacturer" "UNI-ROYAL" (at 182.88 127.0 0) (effects (font (size 1.27 1.27)) hide))
     (pin "1")
     (pin "2")
@@
     (property "Footprint" "Capacitor_SMD:C_0603_1608Metric" (at 71.12 154.94 0) (effects (font (size 1.27 1.27)) hide))
     (property "Datasheet" "~" (at 71.12 154.94 0) (effects (font (size 1.27 1.27)) hide))
+    (property "LCSC" "C14663" (at 71.12 154.94 0) (effects (font (size 1.27 1.27)) hide))
+    (property "MPN" "CC0603KRX7R9BB104" (at 71.12 154.94 0) (effects (font (size 1.27 1.27)) hide))
+    (property "Manufacturer" "YAGEO" (at 71.12 154.94 0) (effects (font (size 1.27 1.27)) hide))
     (pin "1")
     (pin "2")
@@
     (property "Footprint" "Resistor_SMD:R_0603_1608Metric" (at 218.44 88.9 0) (effects (font (size 1.27 1.27)) hide))
     (property "Datasheet" "~" (at 218.44 88.9 0) (effects (font (size 1.27 1.27)) hide))
+    (property "LCSC" "C861257" (at 218.44 88.9 0) (effects (font (size 1.27 1.27)) hide))
+    (property "MPN" "RT0603BRD0725K5L" (at 218.44 88.9 0) (effects (font (size 1.27 1.27)) hide))
+    (property "Manufacturer" "YAGEO" (at 218.44 88.9 0) (effects (font (size 1.27 1.27)) hide))
     (pin "1")
     (pin "2")
@@
     (property "Footprint" "Resistor_SMD:R_0603_1608Metric" (at 218.44 106.68 0) (effects (font (size 1.27 1.27)) hide))
     (property "Datasheet" "~" (at 218.44 106.68 0) (effects (font (size 1.27 1.27)) hide))
-    (pin "1")
-    (pin "2")
+    (property "LCSC" "C110776" (at 218.44 106.68 0) (effects (font (size 1.27 1.27)) hide))
+    (property "MPN" "RT0603BRD071KL" (at 218.44 106.68 0) (effects (font (size 1.27 1.27)) hide))
+    (property "Manufacturer" "YAGEO" (at 218.44 106.68 0) (effects (font (size 1.27 1.27)) hide))
+    (pin "1")
+    (pin "2")
