File: hardware/phase1-module/sensing.kicad_sch (KiCad schematic)
At the start: 11 parts, among them U4 INA240A3, U5 INA228

Commit message: Add LCSC part numbers to all four boards' schematics and generate BOMs
common/bom.py writes hidden LCSC/MPN/Manufacturer properties into the
placed symbols (additive only, both one-line and KiCad multi-line
property styles) and emits <board>/bom/<board>-bom.csv plus a
JLCPCB-format CSV. Part table in common/lcsc_parts.py, transcribed
from SOURCING.md with explicit references per board; CHECK notes flag
footprint/variant mismatches. --check fails on stale output.

Co-Authored-By: Claude Opus 5.5 (1M context) <noreply@anthropic.com>
Claude-Session: https://claude.ai/code/session_01MKtKgebN9BpUrgqHq9t7pT
Parts:
- R30: LCSC (none) -> C2994640
- U4: LCSC (none) -> C2060584; MPN (none) -> INA240A3DR; Manufacturer (none) -> TI
- U5: LCSC (none) -> C2887910; MPN (none) -> INA228AIDGSR; Manufacturer (none) -> TI
Changed lines of the file:
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@@
     (property "Footprint" "Resistor_SMD:R_2512_6332Metric" (at 101.6 55.88 0) (effects (font (size 1.27 1.27)) hide))
     (property "Datasheet" "~" (at 101.6 55.88 0) (effects (font (size 1.27 1.27)) hide))
+    (property "LCSC" "C2994640" (at 101.6 55.88 0) (effects (font (size 1.27 1.27)) hide))
     (pin "1")
     (pin "2")
@@
     (property "Footprint" "Package_SO:SOIC-8_3.9x4.9mm_P1.27mm" (at 76.2 101.6 0) (effects (font (size 1.27 1.27)) hide))
     (property "Datasheet" "~" (at 76.2 101.6 0) (effects (font (size 1.27 1.27)) hide))
+    (property "LCSC" "C2060584" (at 76.2 101.6 0) (effects (font (size 1.27 1.27)) hide))
+    (property "MPN" "INA240A3DR" (at 76.2 101.6 0) (effects (font (size 1.27 1.27)) hide))
+    (property "Manufacturer" "TI" (at 76.2 101.6 0) (effects (font (size 1.27 1.27)) hide))
     (pin "1")
     (pin "2")
@@
     (property "Footprint" "Package_SO:VSSOP-10_3x3mm_P0.5mm" (at 76.2 152.4 0) (effects (font (size 1.27 1.27)) hide))
     (property "Datasheet" "~" (at 76.2 152.4 0) (effects (font (size 1.27 1.27)) hide))
+    (property "LCSC" "C2887910" (at 76.2 152.4 0) (effects (font (size 1.27 1.27)) hide))
+    (property "MPN" "INA228AIDGSR" (at 76.2 152.4 0) (effects (font (size 1.27 1.27)) hide))
+    (property "Manufacturer" "TI" (at 76.2 152.4 0) (effects (font (size 1.27 1.27)) hide))
     (pin "1")
     (pin "10")

Commit message: Phase-1 BOM: LCSC numbers for every assembled part
Fill the 109 missing Phase-1 placements from the JLCPCB catalogue
(checked 2026-09-27, Basic parts where one fits), so 127 of 136
placements carry an LCSC number. J1-J6 and F1 stay hand-solder;
C17 and R17 are DNP.

Out-of-stock swaps: Q1-Q4 CSD18563Q5A -> NTMFS5C670NLT1G (SO-8FL,
same pinout), P1 U5 INA228AIDGSR -> INA228AQDGSRQ1. Y1 moves to the
CL = 12 pF version of the same crystal (C400090 was the 10 pF one).

Co-Authored-By: Claude Opus 5.5 (1M context) <noreply@anthropic.com>
Claude-Session: https://claude.ai/code/session_013uVohQZFdivAh43gw4mZtf
Parts:
- C31, C32: LCSC (none) -> C1588; MPN (none) -> CL10B102KB8NNNC; Manufacturer (none) -> Samsung Electro-Mechanics
- C33, C34: LCSC (none) -> C14663; MPN (none) -> CC0603KRX7R9BB104; Manufacturer (none) -> YAGEO
- R31: LCSC (none) -> C21190; MPN (none) -> 0603WAF1001T5E; Manufacturer (none) -> UNI-ROYAL
- R32: LCSC (none) -> C861526; MPN (none) -> RT0603BRD0769K8L; Manufacturer (none) -> YAGEO
- R33: LCSC (none) -> C95204; MPN (none) -> RT0603BRD0710KL; Manufacturer (none) -> YAGEO
- U5: LCSC C2887910 -> C5214669; MPN INA228AIDGSR -> INA228AQDGSRQ1
Changed lines of the file:
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@@
     (property "Footprint" "Resistor_SMD:R_0603_1608Metric" (at 104.14 96.52 0) (effects (font (size 1.27 1.27)) hide))
     (property "Datasheet" "~" (at 104.14 96.52 0) (effects (font (size 1.27 1.27)) hide))
+    (property "LCSC" "C21190" (at 104.14 96.52 0) (effects (font (size 1.27 1.27)) hide))
+    (property "MPN" "0603WAF1001T5E" (at 104.14 96.52 0) (effects (font (size 1.27 1.27)) hide))
+    (property "Manufacturer" "UNI-ROYAL" (at 104.14 96.52 0) (effects (font (size 1.27 1.27)) hide))
     (pin "1")
     (pin "2")
@@
     (property "Footprint" "Capacitor_SMD:C_0603_1608Metric" (at 118.11 106.68 0) (effects (font (size 1.27 1.27)) hide))
     (property "Datasheet" "~" (at 118.11 106.68 0) (effects (font (size 1.27 1.27)) hide))
+    (property "LCSC" "C1588" (at 118.11 106.68 0) (effects (font (size 1.27 1.27)) hide))
+    (property "MPN" "CL10B102KB8NNNC" (at 118.11 106.68 0) (effects (font (size 1.27 1.27)) hide))
+    (property "Manufacturer" "Samsung Electro-Mechanics" (at 118.11 106.68 0) (effects (font (size 1.27 1.27)) hide))
     (pin "1")
     (pin "2")
@@
     (property "Footprint" "Capacitor_SMD:C_0603_1608Metric" (at 55.88 106.68 0) (effects (font (size 1.27 1.27)) hide))
     (property "Datasheet" "~" (at 55.88 106.68 0) (effects (font (size 1.27 1.27)) hide))
+    (property "LCSC" "C14663" (at 55.88 106.68 0) (effects (font (size 1.27 1.27)) hide))
+    (property "MPN" "CC0603KRX7R9BB104" (at 55.88 106.68 0) (effects (font (size 1.27 1.27)) hide))
+    (property "Manufacturer" "YAGEO" (at 55.88 106.68 0) (effects (font (size 1.27 1.27)) hide))
     (pin "1")
     (pin "2")
@@
     (property "Footprint" "Package_SO:VSSOP-10_3x3mm_P0.5mm" (at 76.2 152.4 0) (effects (font (size 1.27 1.27)) hide))
     (property "Datasheet" "~" (at 76.2 152.4 0) (effects (font (size 1.27 1.27)) hide))
-    (property "LCSC" "C2887910" (at 76.2 152.4 0) (effects (font (size 1.27 1.27)) hide))
-    (property "MPN" "INA228AIDGSR" (at 76.2 152.4 0) (effects (font (size 1.27 1.27)) hide))
+    (property "LCSC" "C5214669" (at 76.2 152.4 0) (effects (font (size 1.27 1.27)) hide))
+    (property "MPN" "INA228AQDGSRQ1" (at 76.2 152.4 0) (effects (font (size 1.27 1.27)) hide))
     (property "Manufacturer" "TI" (at 76.2 152.4 0) (effects (font (size 1.27 1.27)) hide))
     (pin "1")
@@
     (property "Footprint" "Capacitor_SMD:C_0603_1608Metric" (at 55.88 157.48 0) (effects (font (size 1.27 1.27)) hide))
     (property "Datasheet" "~" (at 55.88 157.48 0) (effects (font (size 1.27 1.27)) hide))
+    (property "LCSC" "C14663" (at 55.88 157.48 0) (effects (font (size 1.27 1.27)) hide))
+    (property "MPN" "CC0603KRX7R9BB104" (at 55.88 157.48 0) (effects (font (size 1.27 1.27)) hide))
+    (property "Manufacturer" "YAGEO" (at 55.88 157.48 0) (effects (font (size 1.27 1.27)) hide))
     (pin "1")
     (pin "2")
@@
     (property "Footprint" "Resistor_SMD:R_0603_1608Metric" (at 165.1 88.9 0) (effects (font (size 1.27 1.27)) hide))
     (property "Datasheet" "~" (at 165.1 88.9 0) (effects (font (size 1.27 1.27)) hide))
+    (property "LCSC" "C861526" (at 165.1 88.9 0) (effects (font (size 1.27 1.27)) hide))
+    (property "MPN" "RT0603BRD0769K8L" (at 165.1 88.9 0) (effects (font (size 1.27 1.27)) hide))
+    (property "Manufacturer" "YAGEO" (at 165.1 88.9 0) (effects (font (size 1.27 1.27)) hide))
     (pin "1")
     (pin "2")
@@
     (property "Footprint" "Resistor_SMD:R_0603_1608Metric" (at 165.1 104.14 0) (effects (font (size 1.27 1.27)) hide))
     (property "Datasheet" "~" (at 165.1 104.14 0) (effects (font (size 1.27 1.27)) hide))
+    (property "LCSC" "C95204" (at 165.1 104.14 0) (effects (font (size 1.27 1.27)) hide))
+    (property "MPN" "RT0603BRD0710KL" (at 165.1 104.14 0) (effects (font (size 1.27 1.27)) hide))
+    (property "Manufacturer" "YAGEO" (at 165.1 104.14 0) (effects (font (size 1.27 1.27)) hide))
     (pin "1")
     (pin "2")
@@
     (property "Footprint" "Capacitor_SMD:C_0603_1608Metric" (at 180.34 106.68 0) (effects (font (size 1.27 1.27)) hide))
     (property "Datasheet" "~" (at 180.34 106.68 0) (effects (font (size 1.27 1.27)) hide))
+    (property "LCSC" "C1588" (at 180.34 106.68 0) (effects (font (size 1.27 1.27)) hide))
+    (property "MPN" "CL10B102KB8NNNC" (at 180.34 106.68 0) (effects (font (size 1.27 1.27)) hide))
+    (property "Manufacturer" "Samsung Electro-Mechanics" (at 180.34 106.68 0) (effects (font (size 1.27 1.27)) hide))
     (pin "1")
     (pin "2")
