File: hardware/phase1-module/aux-rails.kicad_sch (KiCad schematic)
At the start: 14 parts, among them U8 LMR36015AQRNXRQ1, U9 NCP1117-3.3

Commit message: Add LCSC part numbers to all four boards' schematics and generate BOMs
common/bom.py writes hidden LCSC/MPN/Manufacturer properties into the
placed symbols (additive only, both one-line and KiCad multi-line
property styles) and emits <board>/bom/<board>-bom.csv plus a
JLCPCB-format CSV. Part table in common/lcsc_parts.py, transcribed
from SOURCING.md with explicit references per board; CHECK notes flag
footprint/variant mismatches. --check fails on stale output.

Co-Authored-By: Claude Opus 5.5 (1M context) <noreply@anthropic.com>
Claude-Session: https://claude.ai/code/session_01MKtKgebN9BpUrgqHq9t7pT
Parts:
- U8: LCSC (none) -> C1850345; MPN (none) -> LMR36015ARNXR; Manufacturer (none) -> TI
- U9: LCSC (none) -> C26537; MPN (none) -> NCP1117ST33T3G; Manufacturer (none) -> onsemi
Changed lines of the file:
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@@
     (property "Footprint" "labbench:LMR36015_RNX_VQFN-HR-12" (at 76.2 78.74 0) (effects (font (size 1.27 1.27)) hide))
     (property "Datasheet" "~" (at 76.2 78.74 0) (effects (font (size 1.27 1.27)) hide))
+    (property "LCSC" "C1850345" (at 76.2 78.74 0) (effects (font (size 1.27 1.27)) hide))
+    (property "MPN" "LMR36015ARNXR" (at 76.2 78.74 0) (effects (font (size 1.27 1.27)) hide))
+    (property "Manufacturer" "TI" (at 76.2 78.74 0) (effects (font (size 1.27 1.27)) hide))
     (pin "1")
     (pin "10")
@@
     (property "Footprint" "Package_TO_SOT_SMD:SOT-223-3_TabPin2" (at 177.8 78.74 0) (effects (font (size 1.27 1.27)) hide))
     (property "Datasheet" "~" (at 177.8 78.74 0) (effects (font (size 1.27 1.27)) hide))
-    (pin "1")
-    (pin "2")
+    (property "LCSC" "C26537" (at 177.8 78.74 0) (effects (font (size 1.27 1.27)) hide))
+    (property "MPN" "NCP1117ST33T3G" (at 177.8 78.74 0) (effects (font (size 1.27 1.27)) hide))
+    (property "Manufacturer" "onsemi" (at 177.8 78.74 0) (effects (font (size 1.27 1.27)) hide))
+    (pin "1")
+    (pin "2")

Commit message: Phase-1 BOM: LCSC numbers for every assembled part
Fill the 109 missing Phase-1 placements from the JLCPCB catalogue
(checked 2026-09-27, Basic parts where one fits), so 127 of 136
placements carry an LCSC number. J1-J6 and F1 stay hand-solder;
C17 and R17 are DNP.

Out-of-stock swaps: Q1-Q4 CSD18563Q5A -> NTMFS5C670NLT1G (SO-8FL,
same pinout), P1 U5 INA228AIDGSR -> INA228AQDGSRQ1. Y1 moves to the
CL = 12 pF version of the same crystal (C400090 was the 10 pF one).

Co-Authored-By: Claude Opus 5.5 (1M context) <noreply@anthropic.com>
Claude-Session: https://claude.ai/code/session_013uVohQZFdivAh43gw4mZtf
Parts:
- C50, C51: LCSC (none) -> C596318; MPN (none) -> CC1210KKX7R9BB475; Manufacturer (none) -> YAGEO
- C52: LCSC (none) -> C14663; MPN (none) -> CC0603KRX7R9BB104; Manufacturer (none) -> YAGEO
- C53: LCSC (none) -> C15849; MPN (none) -> CL10A105KB8NNNC; Manufacturer (none) -> Samsung Electro-Mechanics
- C54, C55, C57: LCSC (none) -> C5341638; MPN (none) -> CC1210KKX7R8BB226; Manufacturer (none) -> YAGEO
- C56: LCSC (none) -> C77102; MPN (none) -> GRM32ER71H106KA12L; Manufacturer (none) -> Murata Electronics
- L2: LCSC (none) -> C223226; MPN (none) -> CBC3225T330KR; Manufacturer (none) -> Taiyo Yuden
- R50, R52: LCSC (none) -> C25803; MPN (none) -> 0603WAF1003T5E; Manufacturer (none) -> UNI-ROYAL
- R51: LCSC (none) -> C25962; MPN (none) -> 0603WAF2492T5E; Manufacturer (none) -> UNI-ROYAL
Changed lines of the file:
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@@
     (property "Footprint" "Capacitor_SMD:C_1210_3225Metric" (at 38.1 83.82 0) (effects (font (size 1.27 1.27)) hide))
     (property "Datasheet" "~" (at 38.1 83.82 0) (effects (font (size 1.27 1.27)) hide))
+    (property "LCSC" "C596318" (at 38.1 83.82 0) (effects (font (size 1.27 1.27)) hide))
+    (property "MPN" "CC1210KKX7R9BB475" (at 38.1 83.82 0) (effects (font (size 1.27 1.27)) hide))
+    (property "Manufacturer" "YAGEO" (at 38.1 83.82 0) (effects (font (size 1.27 1.27)) hide))
     (pin "1")
     (pin "2")
@@
     (property "Footprint" "Capacitor_SMD:C_1210_3225Metric" (at 48.26 83.82 0) (effects (font (size 1.27 1.27)) hide))
     (property "Datasheet" "~" (at 48.26 83.82 0) (effects (font (size 1.27 1.27)) hide))
+    (property "LCSC" "C596318" (at 48.26 83.82 0) (effects (font (size 1.27 1.27)) hide))
+    (property "MPN" "CC1210KKX7R9BB475" (at 48.26 83.82 0) (effects (font (size 1.27 1.27)) hide))
+    (property "Manufacturer" "YAGEO" (at 48.26 83.82 0) (effects (font (size 1.27 1.27)) hide))
     (pin "1")
     (pin "2")
@@
     (property "Footprint" "Capacitor_SMD:C_0603_1608Metric" (at 99.06 63.5 0) (effects (font (size 1.27 1.27)) hide))
     (property "Datasheet" "~" (at 99.06 63.5 0) (effects (font (size 1.27 1.27)) hide))
+    (property "LCSC" "C14663" (at 99.06 63.5 0) (effects (font (size 1.27 1.27)) hide))
+    (property "MPN" "CC0603KRX7R9BB104" (at 99.06 63.5 0) (effects (font (size 1.27 1.27)) hide))
+    (property "Manufacturer" "YAGEO" (at 99.06 63.5 0) (effects (font (size 1.27 1.27)) hide))
     (pin "1")
     (pin "2")
@@
     (property "Footprint" "Capacitor_SMD:C_0603_1608Metric" (at 55.88 99.06 0) (effects (font (size 1.27 1.27)) hide))
     (property "Datasheet" "~" (at 55.88 99.06 0) (effects (font (size 1.27 1.27)) hide))
+    (property "LCSC" "C15849" (at 55.88 99.06 0) (effects (font (size 1.27 1.27)) hide))
+    (property "MPN" "CL10A105KB8NNNC" (at 55.88 99.06 0) (effects (font (size 1.27 1.27)) hide))
+    (property "Manufacturer" "Samsung Electro-Mechanics" (at 55.88 99.06 0) (effects (font (size 1.27 1.27)) hide))
     (pin "1")
     (pin "2")
@@
     (property "Footprint" "Inductor_SMD:L_1210_3225Metric" (at 113.03 91.44 0) (effects (font (size 1.27 1.27)) hide))
     (property "Datasheet" "~" (at 113.03 91.44 0) (effects (font (size 1.27 1.27)) hide))
+    (property "LCSC" "C223226" (at 113.03 91.44 0) (effects (font (size 1.27 1.27)) hide))
+    (property "MPN" "CBC3225T330KR" (at 113.03 91.44 0) (effects (font (size 1.27 1.27)) hide))
+    (property "Manufacturer" "Taiyo Yuden" (at 113.03 91.44 0) (effects (font (size 1.27 1.27)) hide))
     (pin "1")
     (pin "2")
@@
     (property "Footprint" "Resistor_SMD:R_0603_1608Metric" (at 127.0 88.9 0) (effects (font (size 1.27 1.27)) hide))
     (property "Datasheet" "~" (at 127.0 88.9 0) (effects (font (size 1.27 1.27)) hide))
+    (property "LCSC" "C25803" (at 127.0 88.9 0) (effects (font (size 1.27 1.27)) hide))
+    (property "MPN" "0603WAF1003T5E" (at 127.0 88.9 0) (effects (font (size 1.27 1.27)) hide))
+    (property "Manufacturer" "UNI-ROYAL" (at 127.0 88.9 0) (effects (font (size 1.27 1.27)) hide))
     (pin "1")
     (pin "2")
@@
     (property "Footprint" "Resistor_SMD:R_0603_1608Metric" (at 127.0 104.14 0) (effects (font (size 1.27 1.27)) hide))
     (property "Datasheet" "~" (at 127.0 104.14 0) (effects (font (size 1.27 1.27)) hide))
+    (property "LCSC" "C25962" (at 127.0 104.14 0) (effects (font (size 1.27 1.27)) hide))
+    (property "MPN" "0603WAF2492T5E" (at 127.0 104.14 0) (effects (font (size 1.27 1.27)) hide))
+    (property "Manufacturer" "UNI-ROYAL" (at 127.0 104.14 0) (effects (font (size 1.27 1.27)) hide))
     (pin "1")
     (pin "2")
@@
     (property "Footprint" "Capacitor_SMD:C_1210_3225Metric" (at 141.0 88.9 0) (effects (font (size 1.27 1.27)) hide))
     (property "Datasheet" "~" (at 141.0 88.9 0) (effects (font (size 1.27 1.27)) hide))
+    (property "LCSC" "C5341638" (at 141.0 88.9 0) (effects (font (size 1.27 1.27)) hide))
+    (property "MPN" "CC1210KKX7R8BB226" (at 141.0 88.9 0) (effects (font (size 1.27 1.27)) hide))
+    (property "Manufacturer" "YAGEO" (at 141.0 88.9 0) (effects (font (size 1.27 1.27)) hide))
     (pin "1")
     (pin "2")
@@
     (property "Footprint" "Capacitor_SMD:C_1210_3225Metric" (at 151.16 88.9 0) (effects (font (size 1.27 1.27)) hide))
     (property "Datasheet" "~" (at 151.16 88.9 0) (effects (font (size 1.27 1.27)) hide))
+    (property "LCSC" "C5341638" (at 151.16 88.9 0) (effects (font (size 1.27 1.27)) hide))
+    (property "MPN" "CC1210KKX7R8BB226" (at 151.16 88.9 0) (effects (font (size 1.27 1.27)) hide))
+    (property "Manufacturer" "YAGEO" (at 151.16 88.9 0) (effects (font (size 1.27 1.27)) hide))
     (pin "1")
     (pin "2")
@@
     (property "Footprint" "Resistor_SMD:R_0603_1608Metric" (at 96.52 99.06 0) (effects (font (size 1.27 1.27)) hide))
     (property "Datasheet" "~" (at 96.52 99.06 0) (effects (font (size 1.27 1.27)) hide))
+    (property "LCSC" "C25803" (at 96.52 99.06 0) (effects (font (size 1.27 1.27)) hide))
+    (property "MPN" "0603WAF1003T5E" (at 96.52 99.06 0) (effects (font (size 1.27 1.27)) hide))
+    (property "Manufacturer" "UNI-ROYAL" (at 96.52 99.06 0) (effects (font (size 1.27 1.27)) hide))
     (pin "1")
     (pin "2")
@@
     (property "Footprint" "Capacitor_SMD:C_1210_3225Metric" (at 163.83 88.9 0) (effects (font (size 1.27 1.27)) hide))
     (property "Datasheet" "~" (at 163.83 88.9 0) (effects (font (size 1.27 1.27)) hide))
+    (property "LCSC" "C77102" (at 163.83 88.9 0) (effects (font (size 1.27 1.27)) hide))
+    (property "MPN" "GRM32ER71H106KA12L" (at 163.83 88.9 0) (effects (font (size 1.27 1.27)) hide))
+    (property "Manufacturer" "Murata Electronics" (at 163.83 88.9 0) (effects (font (size 1.27 1.27)) hide))
     (pin "1")
     (pin "2")
@@
     (property "Footprint" "Capacitor_SMD:C_1210_3225Metric" (at 194.31 88.9 0) (effects (font (size 1.27 1.27)) hide))
     (property "Datasheet" "~" (at 194.31 88.9 0) (effects (font (size 1.27 1.27)) hide))
-    (pin "1")
-    (pin "2")
+    (property "LCSC" "C5341638" (at 194.31 88.9 0) (effects (font (size 1.27 1.27)) hide))
+    (property "MPN" "CC1210KKX7R8BB226" (at 194.31 88.9 0) (effects (font (size 1.27 1.27)) hide))
+    (property "Manufacturer" "YAGEO" (at 194.31 88.9 0) (effects (font (size 1.27 1.27)) hide))
+    (pin "1")
+    (pin "2")

Commit message: Phase-1/2 L2 to the 5x5 mm land; close the last BOM CHECK rows
Phase-1 and phase-2 L2 (33u/1.2A aux-buck inductor) sat on 1210 lands,
and no stocked 1210 33 uH is rated above 0.5 A. Both now use the
manager's part, cjiang FNR5040S330MT (C167973, Isat 1.30 A min), on
L_Changjiang_FNR5040S, as an ECO on each routed board:
- phase-1: L2 at (32.6, 61.25); the SW_AUX diagonal is re-ended on the
  new pad and a 0.4 mm F.Cu 5V0 link joins L2's via to C54's.
- phase-2: L2 at (68.4, 57.45) r270; its SW_AUX and 5V0 vias now sit in
  the pads, the two stubs that reached them are gone, and a 0.3 mm stub
  ties C55's 5V0 via to pad 2.
- common/eco_swap_fp.py does the in-place footprint swap (nets, fields
  and path carried over). sheets_common.py, both gen_board.py PLACEMENT
  tables and the aux-rails sheets carry the change, so a rebuild matches.
- DRC unchanged: phase-1 10 silk warnings, phase-2 19 warnings, 0 errors
  and 0 unconnected on both. Fab zips, BOMs and CPLs regenerated.

The other CHECK rows (stock checked 2026-10-06):
- Phase-1 C20/C75-C77: no 22 uF 50 V 1210 is stocked, so the design
  value is now 10u/50V X7R (~0.3 Vpp input ripple at 8 A, 350 kHz).
- Phase-1 Q1-Q4: CSD18563Q5A still out of stock; NTMFS5C670NLT1G stays.
  Its case 488AA terminals land within 0.14 mm of the TI part's on the
  Q5A land.
- Phase-2 U3: LM5143QRHARQ1 is the LM5143A-Q1, same pin map; RHA0040N
  matches the RHA0040P land (EP 3.3, 0.5 pitch, 5.8 span).

No CHECK row is left in any BOM. INA228AQDGSRQ1 stock is down to 5, now
on the order-early list. README, HANDOVER, SOURCING, the build guide and
the tools READMEs are updated.

Co-Authored-By: Claude Opus 5.5 (1M context) <noreply@anthropic.com>
Claude-Session: https://claude.ai/code/session_01Kap1Vqs6wqd3fshJdnERW7
Parts:
- L2: footprint Inductor_SMD:L_1210_3225Metric -> Inductor_SMD:L_Changjiang_FNR5040S; LCSC C223226 -> C167973; MPN CBC3225T330KR -> FNR5040S330MT; Manufacturer Taiyo Yuden -> cjiang (Changjiang Microelectronics)
Changed lines of the file:
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@@
     (property "Reference" "L2" (at 113.03 87.63 0) (effects (font (size 1.27 1.27))))
     (property "Value" "33u/1.2A" (at 113.03 95.25 0) (effects (font (size 1.27 1.27))))
-    (property "Footprint" "Inductor_SMD:L_1210_3225Metric" (at 113.03 91.44 0) (effects (font (size 1.27 1.27)) hide))
+    (property "Footprint" "Inductor_SMD:L_Changjiang_FNR5040S" (at 113.03 91.44 0) (effects (font (size 1.27 1.27)) hide))
     (property "Datasheet" "~" (at 113.03 91.44 0) (effects (font (size 1.27 1.27)) hide))
-    (property "LCSC" "C223226" (at 113.03 91.44 0) (effects (font (size 1.27 1.27)) hide))
-    (property "MPN" "CBC3225T330KR" (at 113.03 91.44 0) (effects (font (size 1.27 1.27)) hide))
-    (property "Manufacturer" "Taiyo Yuden" (at 113.03 91.44 0) (effects (font (size 1.27 1.27)) hide))
+    (property "LCSC" "C167973" (at 113.03 91.44 0) (effects (font (size 1.27 1.27)) hide))
+    (property "MPN" "FNR5040S330MT" (at 113.03 91.44 0) (effects (font (size 1.27 1.27)) hide))
+    (property "Manufacturer" "cjiang (Changjiang Microelectronics)" (at 113.03 91.44 0) (effects (font (size 1.27 1.27)) hide))
     (pin "1")
     (pin "2")
