File: hardware/phase1-module/phase1-module.kicad_pcb (KiCad board)
At the start: 4 copper layers, 100 x 80 mm, 144 parts, among them J1 VBUS IN, J2 SWD, J3 UART, J4 OUTPUT, J5 BACKPLANE, J6 FAN, Q1 CSD18563Q5A, Q2 CSD18563Q5A, Q3 60V NFET, Q4 60V NFET, Q5 2N7002, Q6 2N7002, Q7 2N7002, Q8 2N7002, Q9 2N7002, U1 DAC80502DRXT, U10 STM32G431CBT6, U11 TCAN1042HGV, U2 OPA2333, U3 LM5145RGYR, U4 INA240A3, U5 INA228, U6 LTC7004, U7 TLV7011DCK, U8 LMR36015AQRNXRQ1, U9 NCP1117-3.3, Y1 8MHz

Commit message: Phase-1/2 L2 to the 5x5 mm land; close the last BOM CHECK rows
Phase-1 and phase-2 L2 (33u/1.2A aux-buck inductor) sat on 1210 lands,
and no stocked 1210 33 uH is rated above 0.5 A. Both now use the
manager's part, cjiang FNR5040S330MT (C167973, Isat 1.30 A min), on
L_Changjiang_FNR5040S, as an ECO on each routed board:
- phase-1: L2 at (32.6, 61.25); the SW_AUX diagonal is re-ended on the
  new pad and a 0.4 mm F.Cu 5V0 link joins L2's via to C54's.
- phase-2: L2 at (68.4, 57.45) r270; its SW_AUX and 5V0 vias now sit in
  the pads, the two stubs that reached them are gone, and a 0.3 mm stub
  ties C55's 5V0 via to pad 2.
- common/eco_swap_fp.py does the in-place footprint swap (nets, fields
  and path carried over). sheets_common.py, both gen_board.py PLACEMENT
  tables and the aux-rails sheets carry the change, so a rebuild matches.
- DRC unchanged: phase-1 10 silk warnings, phase-2 19 warnings, 0 errors
  and 0 unconnected on both. Fab zips, BOMs and CPLs regenerated.

The other CHECK rows (stock checked 2026-10-06):
- Phase-1 C20/C75-C77: no 22 uF 50 V 1210 is stocked, so the design
  value is now 10u/50V X7R (~0.3 Vpp input ripple at 8 A, 350 kHz).
- Phase-1 Q1-Q4: CSD18563Q5A still out of stock; NTMFS5C670NLT1G stays.
  Its case 488AA terminals land within 0.14 mm of the TI part's on the
  Q5A land.
- Phase-2 U3: LM5143QRHARQ1 is the LM5143A-Q1, same pin map; RHA0040N
  matches the RHA0040P land (EP 3.3, 0.5 pitch, 5.8 span).

No CHECK row is left in any BOM. INA228AQDGSRQ1 stock is down to 5, now
on the order-early list. README, HANDOVER, SOURCING, the build guide and
the tools READMEs are updated.

Co-Authored-By: Claude Opus 5.5 (1M context) <noreply@anthropic.com>
Claude-Session: https://claude.ai/code/session_01Kap1Vqs6wqd3fshJdnERW7
Parts:
- C20, C75, C76, C77: value 22u/50V X7R -> 10u/50V X7R
- L2: footprint Inductor_SMD:L_1210_3225Metric -> Inductor_SMD:L_Changjiang_FNR5040S
- moved L2 0.47 mm to (32.6, 61.2)
Routing:
- net SW_AUX: track 28.8 -> 27.6 mm
- net 5V0: track 83.8 -> 84.8 mm
Changed lines of the file:
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@@
     )
   )
+  (footprint "Inductor_SMD:L_Changjiang_FNR5040S" (layer "F.Cu")
+    (at 32.6 61.25)
+    (descr "Inductor, Changjiang, FNR5040S, 5.0x5.0x4.0mm, https://datasheet.lcsc.com/lcsc/1806131217_cjiang-Changjiang-Microelectronics-Tech-FNR5040S3R3NT_C167960.pdf")
+    (tags "Inductor wirewound power shielded")
+    (attr smd)
+    (fp_text reference "L2" (at -3.949999 0) (layer "F.SilkS")
+        (effects (font (size 0.8 0.8) (thickness 0.12)))
+    )
+    (fp_text value "33u/1.2A" (at 0 3.5) (layer "F.Fab")
+        (effects (font (size 1 1) (thickness 0.15)))
+    )
+    (fp_text user "${REFERENCE}" (at 0 0) (layer "F.Fab")
+        (effects (font (size 0.5 0.5) (thickness 0.075)))
+    )
+    (fp_line (start -2.76 -2.76) (end -2.76 -2.36)
+      (stroke (width 0.12) (type solid)) (layer "F.SilkS"))
+    (fp_line (start -2.76 -2.76) (end 2.76 -2.76)
+      (stroke (width 0.12) (type solid)) (layer "F.SilkS"))
+    (fp_line (start -2.76 2.76) (end -2.76 2.36)
+      (stroke (width 0.12) (type solid)) (layer "F.SilkS"))
+    (fp_line (start -2.76 2.76) (end 2.76 2.76)
+      (stroke (width 0.12) (type solid)) (layer "F.SilkS"))
+    (fp_line (start 2.76 -2.76) (end 2.76 -2.36)
+      (stroke (width 0.12) (type solid)) (layer "F.SilkS"))
+    (fp_line (start 2.76 2.76) (end 2.76 2.36)
+      (stroke (width 0.12) (type solid)) (layer "F.SilkS"))
+    (fp_line (start -2.8 -2.75) (end -2.8 2.75)
+      (stroke (width 0.05) (type solid)) (layer "F.CrtYd"))
+    (fp_line (start -2.8 2.75) (end 2.8 2.75)
+      (stroke (width 0.05) (type solid)) (layer "F.CrtYd"))
+    (fp_line (start 2.8 -2.75) (end -2.8 -2.75)
+      (stroke (width 0.05) (type solid)) (layer "F.CrtYd"))
+    (fp_line (start 2.8 2.75) (end 2.8 -2.75)
+      (stroke (width 0.05) (type solid)) (layer "F.CrtYd"))
+    (fp_line (start -2.5 -2.5) (end -2.5 2.5)
+      (stroke (width 0.1) (type solid)) (layer "F.Fab"))
+    (fp_line (start -2.5 2.5) (end 2.5 2.5)
+      (stroke (width 0.1) (type solid)) (layer "F.Fab"))
+    (fp_line (start 2.5 -2.5) (end -2.5 -2.5)
+      (stroke (width 0.1) (type solid)) (layer "F.Fab"))
+    (fp_line (start 2.5 2.5) (end 2.5 -2.5)
+      (stroke (width 0.1) (type solid)) (layer "F.Fab"))
+    (pad "1" smd rect (at -1.85 0) (size 1.4 4.2) (layers "F.Cu" "F.Paste" "F.Mask")
+      (net 76 "SW_AUX"))
+    (pad "2" smd rect (at 1.85 0) (size 1.4 4.2) (layers "F.Cu" "F.Paste" "F.Mask")
+      (net 2 "5V0"))
+    (model "${KICAD7_3DMODEL_DIR}/Inductor_SMD.3dshapes/L_Changjiang_FNR5040S.wrl"
+      (offset (xyz 0 0 0))
+      (scale (xyz 1 1 1))
+      (rotate (xyz 0 0 0))
+    )
+  )
   (footprint "Capacitor_SMD:C_0603_1608Metric" (layer "F.Cu")
     (at 96.7 75.8)
@@
         (effects (font (size 0.8 0.8) (thickness 0.12)))
     )
-    (fp_text value "22u/50V X7R" (at 0 2.3 -90) (layer "F.Fab")
+    (fp_text value "10u/50V X7R" (at 0 2.3 -90) (layer "F.Fab")
         (effects (font (size 1 1) (thickness 0.15)))
     )
@@
         (effects (font (size 0.8 0.8) (thickness 0.12)))
     )
-    (fp_text value "22u/50V X7R" (at 0 2.3 -90) (layer "F.Fab")
+    (fp_text value "10u/50V X7R" (at 0 2.3 -90) (layer "F.Fab")
         (effects (font (size 1 1) (thickness 0.15)))
     )
@@
     )
   )
-  (footprint "Inductor_SMD:L_1210_3225Metric" (layer "F.Cu")
-    (at 33 61)
-    (descr "Inductor SMD 1210 (3225 Metric), square (rectangular) end terminal, IPC_7351 nominal, (Body size source: http://www.tortai-tech.com/upload/download/2011102023233369053.pdf), generated with kicad-footprint-generator")
-    (tags "inductor")
-    (attr smd)
-    (fp_text reference "L2" (at 0 2.279999) (layer "F.SilkS")
-        (effects (font (size 0.8 0.8) (thickness 0.12)))
-    )
-    (fp_text value "33u/1.2A" (at 0 2.28) (layer "F.Fab")
-        (effects (font (size 1 1) (thickness 0.15)))
-    )
-    (fp_text user "${REFERENCE}" (at 0 0) (layer "F.Fab")
-        (effects (font (size 0.8 0.8) (thickness 0.12)))
-    )
-    (fp_line (start -0.602064 -1.36) (end 0.602064 -1.36)
-      (stroke (width 0.12) (type solid)) (layer "F.SilkS"))
-    (fp_line (start -0.602064 1.36) (end 0.602064 1.36)
-      (stroke (width 0.12) (type solid)) (layer "F.SilkS"))
-    (fp_line (start -2.28 -1.58) (end 2.28 -1.58)
-      (stroke (width 0.05) (type solid)) (layer "F.CrtYd"))
-    (fp_line (start -2.28 1.58) (end -2.28 -1.58)
-      (stroke (width 0.05) (type solid)) (layer "F.CrtYd"))
-    (fp_line (start 2.28 -1.58) (end 2.28 1.58)
-      (stroke (width 0.05) (type solid)) (layer "F.CrtYd"))
-    (fp_line (start 2.28 1.58) (end -2.28 1.58)
-      (stroke (width 0.05) (type solid)) (layer "F.CrtYd"))
-    (fp_line (start -1.6 -1.25) (end 1.6 -1.25)
-      (stroke (width 0.1) (type solid)) (layer "F.Fab"))
-    (fp_line (start -1.6 1.25) (end -1.6 -1.25)
-      (stroke (width 0.1) (type solid)) (layer "F.Fab"))
-    (fp_line (start 1.6 -1.25) (end 1.6 1.25)
-      (stroke (width 0.1) (type solid)) (layer "F.Fab"))
-    (fp_line (start 1.6 1.25) (end -1.6 1.25)
-      (stroke (width 0.1) (type solid)) (layer "F.Fab"))
-    (pad "1" smd roundrect (at -1.4 0) (size 1.25 2.65) (layers "F.Cu" "F.Paste" "F.Mask") (roundrect_rratio 0.2)
-      (net 76 "SW_AUX"))
-    (pad "2" smd roundrect (at 1.4 0) (size 1.25 2.65) (layers "F.Cu" "F.Paste" "F.Mask") (roundrect_rratio 0.2)
-      (net 2 "5V0"))
-    (model "${KICAD6_3DMODEL_DIR}/Inductor_SMD.3dshapes/L_1210_3225Metric.wrl"
-      (offset (xyz 0 0 0))
-      (scale (xyz 1 1 1))
-      (rotate (xyz 0 0 0))
-    )
-  )
   (footprint "Capacitor_SMD:C_0603_1608Metric" (layer "F.Cu")
     (at 60.2 64)
@@
         (effects (font (size 0.8 0.8) (thickness 0.12)))
     )
-    (fp_text value "22u/50V X7R" (at 0 2.3 -90) (layer "F.Fab")
+    (fp_text value "10u/50V X7R" (at 0 2.3 -90) (layer "F.Fab")
         (effects (font (size 1 1) (thickness 0.15)))
     )
@@
         (effects (font (size 0.8 0.8) (thickness 0.12)))
     )
-    (fp_text value "22u/50V X7R" (at 0 2.3 -90) (layer "F.Fab")
+    (fp_text value "10u/50V X7R" (at 0 2.3 -90) (layer "F.Fab")
         (effects (font (size 1 1) (thickness 0.15)))
     )
@@
   (segment (start 87.9888 64.2) (end 87.5888 64.599999) (width 0.2) (layer "F.Cu") (net 2))
   (segment (start 96.0888 64.2) (end 96.1 64.2) (width 0.2) (layer "F.Cu") (net 2))
+  (segment (start 35.5 61) (end 36.425 61) (width 0.4) (layer "F.Cu") (net 2))
   (segment (start 117.95 60.1) (end 117.95 60.55) (width 0.25) (layer "F.Cu") (net 2))
   (segment (start 108.225 76.3) (end 107.125 76.3) (width 0.4) (layer "F.Cu") (net 2))
@@
   (segment (start 36.693 52.9976) (end 37.0023 52.9976) (width 0.2) (layer "F.Cu") (net 76))
   (segment (start 33 54.212) (end 33 52.9976) (width 0.2) (layer "F.Cu") (net 76))
-  (segment (start 28.35 57.75) (end 31.6 61) (width 0.2) (layer "F.Cu") (net 76))
+  (segment (start 28.35 57.75) (end 30.75 60.15) (width 0.2) (layer "F.Cu") (net 76))
   (segment (start 36.7226 52.9976) (end 36.693 52.9976) (width 0.2) (layer "F.Cu") (net 76))
   (segment (start 29.0895 50.5336) (end 28.35 51.2731) (width 0.2) (layer "F.Cu") (net 76))
