File: hardware/phase3-manager/ui.kicad_sch (KiCad schematic)
At the start: 41 parts, among them J5 PANEL KEYS, J6 ILI9341 LCD MODULE, Q10 2N7002, Q11 AO3401A-class PMOS, Q9 2N7002, U13 TCA9535PWR

Commit message: Apply China-sourcing engineering changes across all boards + mechanical frame
All datasheet-verified before application (details hardware/SOURCING.md sF):
- TMUX1101 -> TS5A3166DBVR (LCSC availability; ts5a3166.pdf: pin POSITIONS
  identical - 1=NO 2=COM 3=GND 4=IN 5=V+; VIH 2.4V ok from 3.3V GPIO)
- TLV7011 DBVR -> DCKR: tlv7022.pdf shows DBV/DCK share one pinout, so
  footprint-only (SOT-353_SC-70-5); SOT-23-5 stock in China is nearly gone
- crystal load caps 10p -> 18p, both phases (CL=12pF China crystals; the
  HANDOVER-blessed alternative to hunting CL=8pF parts)
- Phase-1 inductor -> MWSA1707S-100MT (JLCPCB-verified 16.5A Isat/10.5A
  Irms vs 12A/8A required); value strings now dual-source Sunlord/Coilcraft
- module slot power + P2 output -> XT60PW-M (2-pin), backplane slots ->
  XT60PW-F; bus shunt -> 2x BVS-M-R0005 parallel (the exact-net checker
  caught RS1/RS2 placed one pin-span apart merging VBUS_IN into VBUS)
- 470u bulk -> THT radial D10; output MLCCs 22u -> 10u/50V X7S; buzzer ->
  MLT-8530 (fp placeholder)
All four checker chains green: 137/173/30/80 components.

hardware/MECHANICAL.md (frozen): 30mm slot pitch, P2 130x90 4-layer,
backplane ~330x100 2-layer 2oz, manager 100x80; cost-first stackup (1oz
outer + solder-reinforced bus, 2oz only if the thermal soak demands it);
inductor footprint = SUPERSET pattern accepting Sunlord 1707 AND Coilcraft
XAL1510 so the A/B pair is a pure part swap.

HANDOVER: sub-0.5V mV-accurate output DEFERRED to a future dedicated
linear post-regulator module (user decision 2026-07-18); buck floors
documented (P2 0.7V @30V bus, P1 0.5V).

Co-Authored-By: Claude Fable 5 <noreply@anthropic.com>
Parts:
- BZ1: value magnetic 5V -> MLT-8530
Changed lines of the file:
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@@
     (in_bom yes) (on_board yes) (dnp no)
     (property "Reference" "BZ1" (at 254.0 133.35 0) (effects (font (size 1.27 1.27)) (justify left)))
-    (property "Value" "magnetic 5V" (at 254.0 135.89000000000001 0) (effects (font (size 1.27 1.27)) (justify left)))
+    (property "Value" "MLT-8530" (at 254.0 135.89000000000001 0) (effects (font (size 1.27 1.27)) (justify left)))
     (property "Footprint" "Buzzer_Beeper:MagneticBuzzer_CUI_CST-931RP-A" (at 254.0 137.16 0) (effects (font (size 1.27 1.27)) hide))
     (property "Datasheet" "~" (at 254.0 137.16 0) (effects (font (size 1.27 1.27)) hide))

Commit message: Footprint pass: China-part land patterns generated, placeholders retired
build_fplib.py sourcing_footprints() - geometry vetted from LCSC/EasyEDA
library pulls (easyeda2kicad), encoded in code like the PowerFET precedent
so regeneration needs no network:
- XT60PW-M / XT60PW-F: power pins 3.8mm pads / 2.9-2.8mm drills @ 7.2mm
  pitch + 0.6x1.6 retention slots. The -F library pull had the RETENTION
  LEGS numbered as pads 1,2 - power pads renumbered to 1,2 to match the -M
  and the Conn_01x02 symbol (a trap no netlist check would ever catch)
- L_1707_XAL1510: SUPERSET pad 5.39x13.2 @ +/-6.405 covering Sunlord
  MWSA1707S (3.5x12.8 @ 7.35) and Coilcraft XAL1510 (3.18x13.2 @ 5.3) -
  the A/B thermal pair and the P1 10uH are pure part swaps
- R3920_BVS bar shunt, MLT-8530 buzzer (edge pads paired 1,1/2,2)
Generators swapped off placeholders (P1 L1, P2 L1/L3/J1/J4, backplane
slots+RS pair, manager buzzer); all four chains green (137/173/30/80).

MECHANICAL.md: insertion geometry corrected to server-PSU style (vertical
rear backplane, modules slide horizontally; XT60 height stagger = power-
first mating). HARD GATE added: XT60 +/- pad mating is ASSUMED until a
mated pair is buzzed out on arrival - required before gerber submission.

Co-Authored-By: Claude Fable 5 <noreply@anthropic.com>
Parts:
- BZ1: footprint Buzzer_Beeper:MagneticBuzzer_CUI_CST-931RP-A -> labbench:MLT-8530
Changed lines of the file:
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@@
     (property "Reference" "BZ1" (at 254.0 133.35 0) (effects (font (size 1.27 1.27)) (justify left)))
     (property "Value" "MLT-8530" (at 254.0 135.89000000000001 0) (effects (font (size 1.27 1.27)) (justify left)))
-    (property "Footprint" "Buzzer_Beeper:MagneticBuzzer_CUI_CST-931RP-A" (at 254.0 137.16 0) (effects (font (size 1.27 1.27)) hide))
+    (property "Footprint" "labbench:MLT-8530" (at 254.0 137.16 0) (effects (font (size 1.27 1.27)) hide))
     (property "Datasheet" "~" (at 254.0 137.16 0) (effects (font (size 1.27 1.27)) hide))
     (pin "1")

Commit message: Add LCSC part numbers to all four boards' schematics and generate BOMs
common/bom.py writes hidden LCSC/MPN/Manufacturer properties into the
placed symbols (additive only, both one-line and KiCad multi-line
property styles) and emits <board>/bom/<board>-bom.csv plus a
JLCPCB-format CSV. Part table in common/lcsc_parts.py, transcribed
from SOURCING.md with explicit references per board; CHECK notes flag
footprint/variant mismatches. --check fails on stale output.

Co-Authored-By: Claude Opus 5.5 (1M context) <noreply@anthropic.com>
Claude-Session: https://claude.ai/code/session_01MKtKgebN9BpUrgqHq9t7pT
Parts:
- BZ1: LCSC (none) -> C94599; MPN (none) -> MLT-8530
- ENC1: LCSC (none) -> C2831776
- U13: LCSC (none) -> C130204; MPN (none) -> TCA9535PWR; Manufacturer (none) -> TI
Changed lines of the file:
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@@
     (property "Footprint" "Package_SO:TSSOP-24_4.4x7.8mm_P0.65mm" (at 63.5 96.52 0) (effects (font (size 1.27 1.27)) hide))
     (property "Datasheet" "~" (at 63.5 96.52 0) (effects (font (size 1.27 1.27)) hide))
+    (property "LCSC" "C130204" (at 63.5 96.52 0) (effects (font (size 1.27 1.27)) hide))
+    (property "MPN" "TCA9535PWR" (at 63.5 96.52 0) (effects (font (size 1.27 1.27)) hide))
+    (property "Manufacturer" "TI" (at 63.5 96.52 0) (effects (font (size 1.27 1.27)) hide))
     (pin "1")
     (pin "10")
@@
     (property "Footprint" "Rotary_Encoder:RotaryEncoder_Alps_EC11E-Switch_Vertical_H20mm" (at 63.5 172.72 0) (effects (font (size 1.27 1.27)) hide))
     (property "Datasheet" "~" (at 63.5 172.72 0) (effects (font (size 1.27 1.27)) hide))
+    (property "LCSC" "C2831776" (at 63.5 172.72 0) (effects (font (size 1.27 1.27)) hide))
     (pin "A")
     (pin "B")
@@
     (property "Footprint" "labbench:MLT-8530" (at 254.0 137.16 0) (effects (font (size 1.27 1.27)) hide))
     (property "Datasheet" "~" (at 254.0 137.16 0) (effects (font (size 1.27 1.27)) hide))
-    (pin "1")
-    (pin "2")
+    (property "LCSC" "C94599" (at 254.0 137.16 0) (effects (font (size 1.27 1.27)) hide))
+    (property "MPN" "MLT-8530" (at 254.0 137.16 0) (effects (font (size 1.27 1.27)) hide))
+    (pin "1")
+    (pin "2")

Commit message: Fix manager ENC1, F1 and BZ1 part numbers to fit their existing lands
- ENC1: C2831776 was a 100 uF/50 V electrolytic, not an encoder. Now Alps
  EC11E18244A5 (C255515), the EC11E with push switch the footprint is for.
- F1: C3207114 was a 6.35 mm cylindrical fuse clip. The land is a
  direct-solder MINI blade, so F1 is now the 2 A fuse itself, Littelfuse
  0297002.WXNV (C151091). The Phase-1 F1 note is corrected the same way.
- BZ1: MLT-8530 is rated 2.5-4.5 V but runs from 5V0. Now YX-SMD8530P
  (C781886), rated 2-5 V, with the same vendor land and pad-1 (+) corner.

Schematic LCSC/MPN fields and BOM CSVs regenerated with common/bom.py.
No footprint or layout change.

Co-Authored-By: Claude Opus 5.5 (1M context) <noreply@anthropic.com>
Claude-Session: https://claude.ai/code/session_01Ekhw9jYnrfxihP7yvxax5H
Parts:
- BZ1: LCSC C94599 -> C781886; MPN MLT-8530 -> YX-SMD8530P; Manufacturer (none) -> Yuexin
- ENC1: LCSC C2831776 -> C255515; MPN (none) -> EC11E18244A5; Manufacturer (none) -> Alps Alpine
Changed lines of the file:
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@@
     (property "Footprint" "Rotary_Encoder:RotaryEncoder_Alps_EC11E-Switch_Vertical_H20mm" (at 63.5 172.72 0) (effects (font (size 1.27 1.27)) hide))
     (property "Datasheet" "~" (at 63.5 172.72 0) (effects (font (size 1.27 1.27)) hide))
-    (property "LCSC" "C2831776" (at 63.5 172.72 0) (effects (font (size 1.27 1.27)) hide))
+    (property "MPN" "EC11E18244A5" (at 63.5 172.72 0) (effects (font (size 1.27 1.27)) hide))
+    (property "Manufacturer" "Alps Alpine" (at 63.5 172.72 0) (effects (font (size 1.27 1.27)) hide))
+    (property "LCSC" "C255515" (at 63.5 172.72 0) (effects (font (size 1.27 1.27)) hide))
     (pin "A")
     (pin "B")
@@
     (property "Footprint" "labbench:MLT-8530" (at 254.0 137.16 0) (effects (font (size 1.27 1.27)) hide))
     (property "Datasheet" "~" (at 254.0 137.16 0) (effects (font (size 1.27 1.27)) hide))
-    (property "LCSC" "C94599" (at 254.0 137.16 0) (effects (font (size 1.27 1.27)) hide))
-    (property "MPN" "MLT-8530" (at 254.0 137.16 0) (effects (font (size 1.27 1.27)) hide))
-    (pin "1")
-    (pin "2")
+    (property "Manufacturer" "Yuexin" (at 254.0 137.16 0) (effects (font (size 1.27 1.27)) hide))
+    (property "LCSC" "C781886" (at 254.0 137.16 0) (effects (font (size 1.27 1.27)) hide))
+    (property "MPN" "YX-SMD8530P" (at 254.0 137.16 0) (effects (font (size 1.27 1.27)) hide))
+    (pin "1")
+    (pin "2")
