File: hardware/phase3-manager/mcu.kicad_sch (KiCad schematic)
At the start: 14 parts, among them J3 USB-C, J4 UART, SW1 RESET, SW2 BOOT, U10 ESP32-S3-WROOM-1-N8R2, U12 TPD2E001

Commit message: Add LCSC part numbers to all four boards' schematics and generate BOMs
common/bom.py writes hidden LCSC/MPN/Manufacturer properties into the
placed symbols (additive only, both one-line and KiCad multi-line
property styles) and emits <board>/bom/<board>-bom.csv plus a
JLCPCB-format CSV. Part table in common/lcsc_parts.py, transcribed
from SOURCING.md with explicit references per board; CHECK notes flag
footprint/variant mismatches. --check fails on stale output.

Co-Authored-By: Claude Opus 5.5 (1M context) <noreply@anthropic.com>
Claude-Session: https://claude.ai/code/session_01MKtKgebN9BpUrgqHq9t7pT
Parts:
- J3: LCSC (none) -> C165948; MPN (none) -> TYPE-C-31-M-12; Manufacturer (none) -> Korean Hroparts
- U10: LCSC (none) -> C2913204; MPN (none) -> ESP32-S3-WROOM-1-N8R2; Manufacturer (none) -> Espressif
- U12: LCSC (none) -> C150526; MPN (none) -> TPD2E001DRLR; Manufacturer (none) -> TI
Changed lines of the file:
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@@
     (property "Footprint" "RF_Module:ESP32-S3-WROOM-1" (at 88.9 111.76 0) (effects (font (size 1.27 1.27)) hide))
     (property "Datasheet" "~" (at 88.9 111.76 0) (effects (font (size 1.27 1.27)) hide))
+    (property "LCSC" "C2913204" (at 88.9 111.76 0) (effects (font (size 1.27 1.27)) hide))
+    (property "MPN" "ESP32-S3-WROOM-1-N8R2" (at 88.9 111.76 0) (effects (font (size 1.27 1.27)) hide))
+    (property "Manufacturer" "Espressif" (at 88.9 111.76 0) (effects (font (size 1.27 1.27)) hide))
     (pin "1")
     (pin "10")
@@
     (property "Footprint" "Connector_USB:USB_C_Receptacle_GCT_USB4105-xx-A_16P_TopMnt_Horizontal" (at 190.5 96.52 0) (effects (font (size 1.27 1.27)) hide))
     (property "Datasheet" "~" (at 190.5 96.52 0) (effects (font (size 1.27 1.27)) hide))
+    (property "LCSC" "C165948" (at 190.5 96.52 0) (effects (font (size 1.27 1.27)) hide))
+    (property "MPN" "TYPE-C-31-M-12" (at 190.5 96.52 0) (effects (font (size 1.27 1.27)) hide))
+    (property "Manufacturer" "Korean Hroparts" (at 190.5 96.52 0) (effects (font (size 1.27 1.27)) hide))
     (pin "A1")
     (pin "A10")
@@
     (property "Footprint" "Package_TO_SOT_SMD:Texas_R-PDSO-N5_DRL-5" (at 190.5 152.4 0) (effects (font (size 1.27 1.27)) hide))
     (property "Datasheet" "~" (at 190.5 152.4 0) (effects (font (size 1.27 1.27)) hide))
-    (pin "1")
-    (pin "2")
+    (property "LCSC" "C150526" (at 190.5 152.4 0) (effects (font (size 1.27 1.27)) hide))
+    (property "MPN" "TPD2E001DRLR" (at 190.5 152.4 0) (effects (font (size 1.27 1.27)) hide))
+    (property "Manufacturer" "TI" (at 190.5 152.4 0) (effects (font (size 1.27 1.27)) hide))
+    (pin "1")
+    (pin "2")

Commit message: Manager J3: order the GCT USB4105-GF-A that the board is routed for
The manager board's USB breakout is drawn to the USB4105 land, but the BOM
listed the HRO TYPE-C-31-M-12, whose signal pads are 0.3 mm longer and
whose shell stakes sit elsewhere. Dropping it onto the routed board gives
38 DRC errors round J3, so the part follows the copper instead:
USB4105-GF-A, C3020560, held in JLCPCB assembly stock (1.1k) though LCSC
retail shows none. USB4105-GF-A-120 (C5184243, 4.7k) is the backup.

Co-Authored-By: Claude Opus 5.5 (1M context) <noreply@anthropic.com>
Claude-Session: https://claude.ai/code/session_012vqeoXfZfZw2oZCwv9rjfw
Parts:
- J3: LCSC C165948 -> C3020560; MPN TYPE-C-31-M-12 -> USB4105-GF-A; Manufacturer Korean Hroparts -> Global Connector Technology
Changed lines of the file:
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@@
     (property "Footprint" "Connector_USB:USB_C_Receptacle_GCT_USB4105-xx-A_16P_TopMnt_Horizontal" (at 190.5 96.52 0) (effects (font (size 1.27 1.27)) hide))
     (property "Datasheet" "~" (at 190.5 96.52 0) (effects (font (size 1.27 1.27)) hide))
-    (property "LCSC" "C165948" (at 190.5 96.52 0) (effects (font (size 1.27 1.27)) hide))
-    (property "MPN" "TYPE-C-31-M-12" (at 190.5 96.52 0) (effects (font (size 1.27 1.27)) hide))
-    (property "Manufacturer" "Korean Hroparts" (at 190.5 96.52 0) (effects (font (size 1.27 1.27)) hide))
+    (property "LCSC" "C3020560" (at 190.5 96.52 0) (effects (font (size 1.27 1.27)) hide))
+    (property "MPN" "USB4105-GF-A" (at 190.5 96.52 0) (effects (font (size 1.27 1.27)) hide))
+    (property "Manufacturer" "Global Connector Technology" (at 190.5 96.52 0) (effects (font (size 1.27 1.27)) hide))
     (pin "A1")
     (pin "A10")
