File: hardware/phase3-manager/phase3-manager.kicad_pcb (KiCad board)
At the start: 2 copper layers, 100 x 80 mm, 87 parts, among them J1 BACKPLANE, J3 USB-C, J4 UART, J5 PANEL KEYS, J6 ILI9341 LCD MODULE, Q10 2N7002, Q11 AO3401A-class PMOS, Q8 2N7002, Q9 2N7002, SW1 RESET, SW2 BOOT, U10 ESP32-S3-WROOM-1-N8R2, U11 TCAN1042HGV, U12 TPD2E001, U13 TCA9535PWR, U8 LMR36015AQRNXRQ1, U9 NCP1117-3.3

Commit message: Manager L2 and backplane C2: pick stocked parts, re-route L2 as an ECO
Manager L2 (33u/1.2A aux-buck inductor) had a 1210 land, and no stocked
1210 33 uH is rated above 0.5 A. It is now the 5x5 mm cjiang
FNR5040S330MT (C167973: Isat 1.30 A min, Irms 1.20 A min, 0.244 ohm)
on KiCad's L_Changjiang_FNR5040S land.

Board ECO, no full re-route:
- L2 moves to (18.8, 48.4) so its courtyard clears C54, F1 and C50/C51;
  C54/C55 turn 180 so their 5V0 pads line up with L2's 5V0 pad (one
  straight 0.8 mm run) and their PGND pads are tied and dropped to the
  plane west of C55.
- SW_AUX and the 5V0 head are redrawn locked, matching route_critical.py;
  PRESENT1/4-7 are re-routed round the bigger part by finish_routes.py.
- gen_board.py PLACEMENT and route_critical.py ROUTES carry the same
  change, so a full rebuild reproduces it.
- DRC: 0 unconnected, 0 errors, 4 warnings (was 5). Fab zip, BOM, CPL
  regenerated.

Backplane C2 (470u/50V on CP_Elec_16x17.5): Nichicon UCX1H471MNS1MS
(C462700, 16x16.5, 70 mOhm), which fits the existing land; Panasonic
EEEFK1H471AM (C178551) is the fallback. No board change.

Co-Authored-By: Claude Opus 5.5 (1M context) <noreply@anthropic.com>
Claude-Session: https://claude.ai/code/session_016Wr11AqV5ZRbpysgP42oHy
Parts:
- L2: footprint Inductor_SMD:L_1210_3225Metric -> Inductor_SMD:L_Changjiang_FNR5040S
- moved L2 1.79 mm to (38.8, 68.4)
- turned C54 to -90 degrees
- turned C55 to -90 degrees
Routing:
- net PRESENT7: track 73.9 -> 60.2 mm, vias 7 -> 9
- net PRESENT6: track 67.9 -> 58.6 mm, vias 2 -> 6
- net PRESENT1: track 58.9 -> 53.5 mm, vias 5 -> 7
- net PGND: track 68.6 -> 71.9 mm, vias 323 -> 325
- net PRESENT5: track 60.7 -> 57.7 mm, vias 2 -> 6
- net PRESENT4: track 58.9 -> 56.2 mm
- net 5V0: track 209.6 -> 211.4 mm
- net SW_AUX: track 17.2 -> 16.5 mm
